File: hardware/touchpad/touchpad-backups/touchpad_backup.kicad_pcb (KiCad board)
At the start: 2 copper layers, 185 x 125 mm, 187 parts, among them J1 Conn_01x26_MountingPin, J10 Conn_02x03_Odd_Even, J100 Conn_02x03_Odd_Even, J101 Conn_02x03_Odd_Even, J102 Conn_02x03_Odd_Even, J103 Conn_02x03_Odd_Even, J104 Conn_02x03_Odd_Even, J105 Conn_02x03_Odd_Even, J106 Conn_02x03_Odd_Even, J107 Conn_02x03_Odd_Even, J108 Conn_02x03_Odd_Even, J109 Conn_02x03_Odd_Even, J11 Conn_02x03_Odd_Even, J110 Conn_02x03_Odd_Even, J111 Conn_02x03_Odd_Even, J112 Conn_02x03_Odd_Even, J113 Conn_02x03_Odd_Even, J114 Conn_02x03_Odd_Even, J115 Conn_02x03_Odd_Even, J116 Conn_02x03_Odd_Even, J117 Conn_02x03_Odd_Even, J118 Conn_02x03_Odd_Even, J119 Conn_02x03_Odd_Even, J12 Conn_02x03_Odd_Even, J120 Conn_02x03_Odd_Even, J121 Conn_02x03_Odd_Even, J122 Conn_02x03_Odd_Even, J123 Conn_02x03_Odd_Even, J124 Conn_02x03_Odd_Even, J125 Conn_02x03_Odd_Even, J126 Conn_02x03_Odd_Even, J127 Conn_02x03_Odd_Even, J128 Conn_02x03_Odd_Even, J129 Conn_02x03_Odd_Even, J13 Conn_02x03_Odd_Even, J130 Conn_02x03_Odd_Even, J131 Conn_02x03_Odd_Even, J132 Conn_02x03_Odd_Even, J133 Conn_02x03_Odd_Even, J134 Conn_02x03_Odd_Even, J135 Conn_02x03_Odd_Even, J136 Conn_02x03_Odd_Even, J137 Conn_02x03_Odd_Even, J138 Conn_02x03_Odd_Even, J139 Conn_02x03_Odd_Even, J14 Conn_02x03_Odd_Even, J140 Conn_02x03_Odd_Even, J141 Conn_02x03_Odd_Even, J142 Conn_02x03_Odd_Even, J143 Conn_02x03_Odd_Even, J144 Conn_02x03_Odd_Even, J145 Conn_02x03_Odd_Even, J146 Conn_02x03_Odd_Even, J147 Conn_02x03_Odd_Even, J148 Conn_02x03_Odd_Even, J149 Conn_02x03_Odd_Even, J15 Conn_02x03_Odd_Even, J150 Conn_02x03_Odd_Even, J151 Conn_02x03_Odd_Even, J152 Conn_02x03_Odd_Even, J153 Conn_02x03_Odd_Even, J154 Conn_02x03_Odd_Even, J155 Conn_02x03_Odd_Even, J156 Conn_02x03_Odd_Even, J157 Conn_02x03_Odd_Even, J158 Conn_02x03_Odd_Even, J159 Conn_02x03_Odd_Even, J16 Conn_02x03_Odd_Even, J160 Conn_02x03_Odd_Even, J161 Conn_02x03_Odd_Even, J162 Conn_02x03_Odd_Even, J163 Conn_02x03_Odd_Even, J164 Conn_02x03_Odd_Even, J165 Conn_02x03_Odd_Even, J166 Conn_02x03_Odd_Even, J167 Conn_02x03_Odd_Even, J168 Conn_02x03_Odd_Even, J169 Conn_02x03_Odd_Even, J17 Conn_02x03_Odd_Even, J170 Conn_02x03_Odd_Even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

Commit message: fixed stuff
Parts:
- J10, J100, J101, J102, J103, J104, J105, J106, J107, J108, J109, J11, J110, J111, J12, J13, J14, J15, J16, J17, J18, J184, J185, J186, J187, J19, J20, J21, J22, J23, J24, J25, J26, J27, J28, J29, J30, J31, J32, J33, J34, J35, J36, J37, J38, J39, J4, J40, J41, J42, J43, J44, J45, J46, J47, J48, J49, J5, J50, J51, J52, J53, J54, J55, J56, J57, J58, J59, J6, J60, J61, J62, J63, J64, J65, J66, J67, J68, J69, J7, J70, J71, J72, J73, J74, J75, J76, J77, J78, J79, J8, J80, J81, J82, J83, J84, J85, J86, J87, J88, J89, J9, J90, J91, J92, J93, J94, J95, J96, J97, J98, J99: moved to F.Cu
- J112, J113, J114, J115, J116, J117, J118, J119, J120, J121, J122, J123, J124, J125, J126, J127, J128, J129, J130, J131, J132, J133, J134, J135, J136, J137, J138, J139, J140, J141, J142, J143, J144, J145, J146, J147, J148, J149, J150, J151, J152, J153, J154, J155, J156, J157, J158, J159, J160, J161, J162, J163, J164, J165, J166, J167, J168, J169, J170, J171, J172, J173, J174, J175, J176, J177, J178, J179, J180, J181, J182, J183: moved to B.Cu
- moved J114 261.3 mm to (43.5, 190.6)
- moved J118 254.0 mm to (43.5, 184.6)
- moved J122 247.1 mm to (43.5, 178.6)
- moved J126 240.5 mm to (43.5, 172.6)
- moved J115 239.3 mm to (43.5, 171.4)
- moved J130 234.4 mm to (43.5, 166.6)
- moved J119 233.2 mm to (43.5, 165.4)
- moved J134 228.8 mm to (43.5, 160.6)
- moved J123 227.7 mm to (43.5, 159.4)
- moved J138 223.6 mm to (43.5, 154.6)
- moved J127 222.6 mm to (43.5, 153.4)
- moved J183 219.1 mm to (43.5, 69.4)
- moved J142 219.0 mm to (43.5, 148.6)
- moved J131 218.1 mm to (43.5, 147.4)
- moved J179 215.0 mm to (43.5, 75.4)
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Routing:
- net Net-(J116-Pin_6): track 169.4 -> 0.00 mm
- net Net-(J116-Pin_4): track 169.4 -> 0.00 mm
- net Net-(J112-Pin_4): track 169.4 -> 0.00 mm
- net Net-(J4-Pin_4): track 109.4 -> 0.00 mm
- net Net-(J112-Pin_5): track 26.2 -> 24.8 mm
- net Net-(J112-Pin_6): track 1.40 -> 0.00 mm
- net Net-(J6-Pin_4): track 24.8 -> 23.5 mm
- net Net-(J6-Pin_2): track 27.5 -> 26.2 mm
- net Net-(J4-Pin_5): track 26.1 -> 24.8 mm
- net Net-(J112-Pin_3): track 25.7 -> 24.7 mm
- net Net-(J110-Pin_2): track 27.0 -> 26.2 mm
- net Net-(J4-Pin_3): track 25.4 -> 24.7 mm
- net Net-(J6-Pin_6): track 24.8 -> 24.1 mm
- net Net-(J170-Pin_2): track 26.8 -> 26.2 mm
- net Net-(J174-Pin_2): track 26.8 -> 26.2 mm
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