File: hardware/touchpad/touchpad-backups/touchpad_before.kicad_pcb (KiCad board)
At the start: 2 copper layers, 190 x 125 mm, 187 parts, among them J1 Conn_01x26_MountingPin, J10 Conn_02x03_Odd_Even, J100 Conn_02x03_Odd_Even, J101 Conn_02x03_Odd_Even, J102 Conn_02x03_Odd_Even, J103 Conn_02x03_Odd_Even, J104 Conn_02x03_Odd_Even, J105 Conn_02x03_Odd_Even, J106 Conn_02x03_Odd_Even, J107 Conn_02x03_Odd_Even, J108 Conn_02x03_Odd_Even, J109 Conn_02x03_Odd_Even, J11 Conn_02x03_Odd_Even, J110 Conn_02x03_Odd_Even, J111 Conn_02x03_Odd_Even, J112 Conn_02x03_Odd_Even, J113 Conn_02x03_Odd_Even, J114 Conn_02x03_Odd_Even, J115 Conn_02x03_Odd_Even, J116 Conn_02x03_Odd_Even, J117 Conn_02x03_Odd_Even, J118 Conn_02x03_Odd_Even, J119 Conn_02x03_Odd_Even, J12 Conn_02x03_Odd_Even, J120 Conn_02x03_Odd_Even, J121 Conn_02x03_Odd_Even, J122 Conn_02x03_Odd_Even, J123 Conn_02x03_Odd_Even, J124 Conn_02x03_Odd_Even, J125 Conn_02x03_Odd_Even, J126 Conn_02x03_Odd_Even, J127 Conn_02x03_Odd_Even, J128 Conn_02x03_Odd_Even, J129 Conn_02x03_Odd_Even, J13 Conn_02x03_Odd_Even, J130 Conn_02x03_Odd_Even, J131 Conn_02x03_Odd_Even, J132 Conn_02x03_Odd_Even, J133 Conn_02x03_Odd_Even, J134 Conn_02x03_Odd_Even, J135 Conn_02x03_Odd_Even, J136 Conn_02x03_Odd_Even, J137 Conn_02x03_Odd_Even, J138 Conn_02x03_Odd_Even, J139 Conn_02x03_Odd_Even, J14 Conn_02x03_Odd_Even, J140 Conn_02x03_Odd_Even, J141 Conn_02x03_Odd_Even, J142 Conn_02x03_Odd_Even, J143 Conn_02x03_Odd_Even, J144 Conn_02x03_Odd_Even, J145 Conn_02x03_Odd_Even, J146 Conn_02x03_Odd_Even, J147 Conn_02x03_Odd_Even, J148 Conn_02x03_Odd_Even, J149 Conn_02x03_Odd_Even, J15 Conn_02x03_Odd_Even, J150 Conn_02x03_Odd_Even, J151 Conn_02x03_Odd_Even, J152 Conn_02x03_Odd_Even, J153 Conn_02x03_Odd_Even, J154 Conn_02x03_Odd_Even, J155 Conn_02x03_Odd_Even, J156 Conn_02x03_Odd_Even, J157 Conn_02x03_Odd_Even, J158 Conn_02x03_Odd_Even, J159 Conn_02x03_Odd_Even, J16 Conn_02x03_Odd_Even, J160 Conn_02x03_Odd_Even, J161 Conn_02x03_Odd_Even, J162 Conn_02x03_Odd_Even, J163 Conn_02x03_Odd_Even, J164 Conn_02x03_Odd_Even, J165 Conn_02x03_Odd_Even, J166 Conn_02x03_Odd_Even, J167 Conn_02x03_Odd_Even, J168 Conn_02x03_Odd_Even, J169 Conn_02x03_Odd_Even, J17 Conn_02x03_Odd_Even, J170 Conn_02x03_Odd_Even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

Commit message: fixed stuff
Parts:
- moved J10 13.6 mm to (42.2, 187.2)
- moved J102 13.6 mm to (180.2, 187.2)
- moved J106 13.6 mm to (186.2, 187.2)
- moved J110 13.6 mm to (192.2, 187.2)
- moved J14 13.6 mm to (48.2, 187.2)
- moved J18 13.6 mm to (54.2, 187.2)
- moved J186 13.6 mm to (198.2, 187.2)
- moved J22 13.6 mm to (60.2, 187.2)
- moved J26 13.6 mm to (66.2, 187.2)
- moved J30 13.6 mm to (72.2, 187.2)
- moved J34 13.6 mm to (78.2, 187.2)
- moved J38 13.6 mm to (84.2, 187.2)
- moved J42 13.6 mm to (90.2, 187.2)
- moved J46 13.6 mm to (96.2, 187.2)
- moved J50 13.6 mm to (102.2, 187.2)
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Routing:
- net Net-(J114-Pin_2): track 26.8 -> 26.2 mm
- net Net-(J6-Pin_4): track 24.1 -> 23.5 mm
- net Net-(J6-Pin_2): track 26.8 -> 26.2 mm
