File: hardware/board/board.kicad_sch (KiCad schematic)
At the start: 29 parts, among them J1 USB_C_Receptacle, U1 STM32WB55RGVx, Y1 32MHz

Commit message: started schematics
Parts:
- added C16, C20: 0.8pF, symbol Device:C
- added C17, C21: 0.3pF, symbol Device:C
- added C18: 1.5pF, symbol Device:C
- added C19: DNP, symbol Device:C
- added C22, C23, C24, C25: 1uF, Capacitor_SMD:C_0402_1005Metric_Pad0.74x0.62mm_HandSolder, symbol Device:C
- added C44, C45, C46, C47, C48, C49, C50, C51, C52, C53: 100nF, Capacitor_SMD:C_0402_1005Metric, symbol Device:C_Small
- added C54: 72nF, Capacitor_SMD:C_0402_1005Metric, symbol Device:C_Small
- added C55: 10uF, symbol Device:C
- added C56: 1uF, symbol Device:C
- added FB3: 100R, Inductor_SMD:L_0603_1608Metric, symbol Device:FerriteBead_Small
- added J2, J3, J4: Conn_01x26_MountingPin, Connector_FFC-FPC:Hirose_FH12-26S-0.5SH_1x26-1MP_P0.50mm_Horizontal, symbol Connector_Generic_MountingPin:Conn_01x26_MountingPin
- added JP1: ~, Jumper:SolderJumper-2_P1.3mm_Bridged_RoundedPad1.0x1.5mm, symbol Jumper:SolderJumper_2_Bridged
- added L2: 2.7nH, symbol Device:L
- added L3: 3nH, symbol Device:L
- added Q4: ~, DMN313DLT-7:SOT-523-3_L1.6-W0.8-P1.00-LS1.6-BR, symbol DMN313DLT-7:DMN313DLT-7
- added R10, R11, R34, R9: 10K, symbol Device:R
- added R31, R32: 1.5K, symbol Device:R
- added R33: 4.7K, symbol Device:R
- added R5: 0, symbol Device:R
- added R6, R7, R8: DNP, symbol Device:R
- added SW1, SW2, SW3: SW_Push, symbol Switch:SW_Push
- added U11, U12, U7, U8 (x2), U9: 74HC4051, Package_DFN_QFN:DHVQFN-16-1EP_2.5x3.5mm_P0.5mm_EP1x2mm, symbol 74xx:74HC4051
- added U2: ~, BQ25896RTWR:QFN-24_L4.0-W4.0-P0.50-TL-EP2.7, symbol BQ25896RTWR:BQ25896RTWR
- added U3: ~, RS3221-3.3YF3:SOT-23-3_L2.9-W1.6-P1.90-LS2.8-BR, symbol RS3221-3.3YF3:RS3221-3.3YF3
- added U4: ~, BQ27220YZFR:DSBGA-9_L1.7-W1.6-R3-C3-P0.50-BL, symbol BQ27220YZFR:BQ27220YZFR
- added U5: ~, COS8054TR:TSSOP-14_L5.0-W4.4-P0.65-LS6.4-BL, symbol COS8054TR:COS8054TR
- added Y2: 32.768kHz, symbol Device:Crystal
Connections:
- net +3.3V: now also R11.1, R31.2, R32.2, R33.2, R9.1
- net GND: now also AE1.1 (A), FLT1.2 (GND), FLT1.5 (GND), C16.2, C17.2, C18.2, C19.1, C19.2, C20.2, C21.2, C55.2, C56.2, FB3.1, J2.14 (Pin_14), J2.19 (Pin_19), J2.24 (Pin_24), J2.4 (Pin_4), J2.9 (Pin_9), J3.14 (Pin_14), J3.19 (Pin_19), J3.24 (Pin_24), J3.4 (Pin_4), J3.9 (Pin_9), J4.14 (Pin_14), J4.19 (Pin_19), J4.24 (Pin_24), J4.4 (Pin_4), J4.9 (Pin_9), L3.2, R10.1, R5.1, R5.2, R6.1, R6.2, R7.1, R7.2, R8.1, R8.2, U2.2 (PSEL)
- net VBUS: now also C44.2, C46.2, C48.2, C50.2, C52.2, U11.16 (VCC), U12.16 (VCC), U7.16 (VCC), U8.16 (VCC), U8.16 (VCC), U9.16 (VCC)
- net BUTTON: now reaches U1.2 (PC13)
- net BUTTON: now also SW3.1
- net I2C_SCL: now reaches U1.24 (PA9)
- net I2C_SCL: now also R31.1, U2.5 (SCL)
- net at U1.3 (PC14): now also C21.1, Y2.2
- net at U1.31 (RF1): now also C16.1, L2.1
- net at U1.4 (PC15): now also C20.1, Y2.1
- net BOOT: now reaches U1.5 (PH3)
- net BOOT: now also SW2.1
- net I2C_SDA: now reaches U1.51 (PA10)
- net I2C_SDA: now also R32.1, U2.6 (SDA)
- net RESET: now reaches U1.8 (NRST)
- net RESET: now also SW1.1
- net at FLT1.1 (IN): now also C17.1, L2.2
- net at FLT1.3 (OUT): now also C18.1, L3.1
- new net: R9.2, SW1.2
- new net: R10.2, SW2.2
- new net: Q4.3 (D), R34.1, U2.8 (OTG)
- new net: R33.1, U2.7 (INT)
- new net: C55.1, U2.23 (PMID)
- new net: R11.2, SW3.2
- new net +5V: C56.1, U2.1 (VBUS)
- new net ABUS: C54.1, U11.3 (A), U12.3 (A), U7.3 (A), U8.3 (A), U8.3 (A), U9.3 (A)
- new net CPH1: C22.1, C23.1
- new net CPH2: C24.1, C25.1
- new net EXCITER: C54.2
- new net GNDS: JP1.1 (A)
- new net S0: U11.11 (S0), U12.11 (S0), U7.11 (S0), U8.11 (S0), U8.11 (S0), U9.11 (S0)
- new net S1: U11.10 (S1), U12.10 (S1), U7.10 (S1), U8.10 (S1), U8.10 (S1), U9.10 (S1)
- new net S2: U11.9 (S2), U12.9 (S2), U7.9 (S2), U8.9 (S2), U8.9 (S2), U9.9 (S2)
- new net TIM8_CH1: C22.2
- new net TIM8_CH3: C23.2
- new net VEE: C45.1, C47.1, C49.1, C51.1, C53.1, JP1.2 (B), U11.7 (VEE), U12.7 (VEE), U7.7 (VEE), U8.7 (VEE), U8.7 (VEE), U9.7 (VEE)
- new net VSSA: C44.1, C45.2, C46.1, C47.2, C48.1, C49.2, C50.1, C51.2, C52.1, C53.2, FB3.2, U11.8 (GND), U12.8 (GND), U7.8 (GND), U8.8 (GND), U8.8 (GND), U9.8 (GND)
- new net X0: J4.26 (Pin_26), U7.13 (A0)
- new net X1: J4.25 (Pin_25), U7.14 (A1)
- new net X10: J4.13 (Pin_13), U8.15 (A2)
- new net X11: J4.12 (Pin_12), U8.12 (A3)
- new net X12: J4.11 (Pin_11), U8.1 (A4)
- new net X13: J4.10 (Pin_10), U8.5 (A5)
- new net X14: J4.8 (Pin_8), U8.2 (A6)
- new net X15: J4.7 (Pin_7), U8.4 (A7)
- new net X16: J4.6 (Pin_6), U9.13 (A0)
- new net X17: J4.5 (Pin_5), U9.14 (A1)
- new net X18: J4.3 (Pin_3), U9.15 (A2)
- new net X19: J4.2 (Pin_2), U9.12 (A3)
- new net X2: J4.23 (Pin_23), U7.15 (A2)
- new net X20: J3.26 (Pin_26), U9.1 (A4)
- new net X21: J3.25 (Pin_25), U9.5 (A5)
- new net X22: J3.23 (Pin_23), U9.2 (A6)
- new net X23: J3.22 (Pin_22), U9.4 (A7)
- new net X24: J3.21 (Pin_21), U8.13 (A0)
- new net X25: J3.20 (Pin_20), U8.14 (A1)
- new net X26: J3.18 (Pin_18), U8.15 (A2)
- new net X27: J3.17 (Pin_17), U8.12 (A3)
- new net X3: J4.22 (Pin_22), U7.12 (A3)
- new net X4: J4.21 (Pin_21), U7.1 (A4)
- new net X5: J4.20 (Pin_20), U7.5 (A5)
- new net X6: J4.18 (Pin_18), U7.2 (A6)
- new net X7: J4.17 (Pin_17), U7.4 (A7)
- new net X8: J4.16 (Pin_16), U8.13 (A0)
- new net X9: J4.15 (Pin_15), U8.14 (A1)
- new net Y0: J2.26 (Pin_26), U8.1 (A4)
- new net Y1: J2.25 (Pin_25), U8.5 (A5)
- new net Y10: J2.13 (Pin_13), U11.2 (A6)
- new net Y11: J2.12 (Pin_12), U11.4 (A7)
- new net Y12: J2.11 (Pin_11), U12.13 (A0)
- new net Y13: J2.10 (Pin_10), U12.14 (A1)
- new net Y14: J2.8 (Pin_8), U12.15 (A2)
- new net Y15: J2.7 (Pin_7), U12.12 (A3)
- new net Y16: J2.6 (Pin_6), U12.1 (A4)
- new net Y17: J2.5 (Pin_5), U12.5 (A5)
- new net Y2: J2.23 (Pin_23), U8.2 (A6)
- new net Y3: J2.22 (Pin_22), U8.4 (A7)
- new net Y4: J2.21 (Pin_21), U11.13 (A0)
- new net Y5: J2.20 (Pin_20), U11.14 (A1)
- new net Y6: J2.18 (Pin_18), U11.15 (A2)
- new net Y7: J2.17 (Pin_17), U11.12 (A3)
- new net Y8: J2.16 (Pin_16), U11.1 (A4)
- new net Y9: J2.15 (Pin_15), U11.5 (A5)
- new net ~{E0}: U7.6 (~{E})
- new net ~{E1}: U8.6 (~{E})
- new net ~{E2}: U9.6 (~{E})
- new net ~{E3}: U8.6 (~{E})
- new net ~{E4}: U11.6 (~{E})
- new net ~{E5}: U12.6 (~{E})
- new net ~{TIM8_CH1}: C24.2
- new net ~{TIM8_CH3}: C25.2
- no-connect marks 10 -> 34
Other:
- added sheet Signal Chain (analog.kicad_sch)
- moved on the sheet: AE1, C15, FLT1, L1

Commit message: update schmatic
Parts:
- removed U5: ~, COS8054TR:TSSOP-14_L5.0-W4.4-P0.65-LS6.4-BL, symbol COS8054TR:COS8054TR
- added C57, C69: 4.7uF, symbol Device:C
- added C58: 47uF, symbol Device:C
- added C59, C60, C61, C62, C70, C71: 10uF, symbol Device:C
- added C63, C67, C68: 2.2uF, symbol Device:C
- added C64: 470nF, symbol Device:C
- added C65, C66: 1uF, symbol Device:C
- added C72: 120pF, Capacitor_SMD:C_0402_1005Metric, symbol Device:C_Small
- added C73: 72nF, Capacitor_SMD:C_0402_1005Metric, symbol Device:C_Small
- added C74: 100nF, Capacitor_SMD:C_0402_1005Metric, symbol Device:C_Small
- added C75: 1uF, Capacitor_SMD:C_0402_1005Metric, symbol Device:C_Small
- added D12: BAT54SW, Package_TO_SOT_SMD:SOT-323_SC-70, symbol Diode:BAT54SW
- added FB5: 100R, Inductor_SMD:L_0603_1608Metric, symbol Device:FerriteBead_Small
- added J5: Conn_01x03, symbol Connector_Generic:Conn_01x03
- added L4: 1uH, symbol Device:L
- added L5, L6: 470nH, symbol Device:L
- added L7: 60R / Short, Inductor_SMD:L_0603_1608Metric, symbol Device:L_Ferrite_Small
- added Q5: ~, MMDT2907A-7-F:SOT-363_L2.0-W1.3-P0.65-LS2.1-BL, symbol MMDT2907A-7-F:MMDT2907A-7-F
- added Q6: ~, DMP1045U-7:SOT-23-3_L2.9-W1.3-P1.90-LS2.4-BR, symbol DMP1045U-7:DMP1045U-7
- added R35: 100, symbol Device:R
- added R36, R40, R41: 10K, symbol Device:R
- added R37: 470, symbol Device:R
- added R38: 30.1K, symbol Device:R
- added R39: 5.23K, symbol Device:R
- added R42: 10m, symbol Device:R
- added R43: DNP, symbol Device:R
- added R44, R45: 1.5, symbol Device:R
- added R46, R47: 3.3, symbol Device:R
- added R48, R49: 100K, symbol Device:R
- added R50: 10k, Resistor_SMD:R_0402_1005Metric, symbol Device:R_Small_US
- added R51: 400, Resistor_SMD:R_0402_1005Metric, symbol Device:R_Small_US
- added U15: SN74LV1T125DCK, Package_TO_SOT_SMD:SOT-353_SC-70-5, symbol Logic_LevelTranslator:SN74LV1T125DCK
- added U5: ~, LM3281YFQR:DSBGA-6_L1.4-W1.1-R3-C2-P0.40-BL, symbol LM3281YFQR:LM3281YFQR
Connections:
- net +3.3V: now also C71.1, R40.2, R46.1, R47.1
- net +5V: now also Q5.4 (E2), Q6.2 (S)
- net ABUS: now also L7.2
- net EXCITER: now also R51.1
- net GND: now also Q4.2 (S), U2.17 (PGND), U2.18 (PGND), U2.25 (EPAD), U2.9 (CE), U3.1 (GND), U4.B2 (VSS), C57.2, C59.2, C60.2, C61.2, C62.2, C63.2, C64.2, C65.2, C66.2, C67.2, C68.2, C69.2, C70.2, C71.2, J5.3 (Pin_3), R36.1, R37.1, R38.1, R41.1, R43.2, R48.2, R49.2, U5.C2 (GND)
- net I2C_SCL: now also U4.A3 (SCL)
- net I2C_SDA: now also U4.A2 (SDA)
- net LDO_3.3V: now also U3.2 (VOUT)
- net RESET: now also U2.12 (QON)
- net VBUS: now also FB5.2, Q5.1 (E1), Q5.2 (B1), Q5.3 (C2), Q5.5 (B2), Q6.3 (D), R35.2, R48.1
- net VSSA: now also C72.1, C74.2, C75.2, U15.3 (GND)
- net at U3.3 (VIN): now also U2.13 (BAT), U2.14 (BAT), U4.C2 (SRN), C61.1, C62.1, C66.1, R42.2
- net at Q4.1 (G): now also R35.1, R36.2
- net SYS: now reaches R34.2
- net SYS: now also U2.15 (SYS), U2.16 (SYS), C59.1, C60.1, C67.1, L4.2, U5.A2 (VIN), U5.B1 (MODE), U5.C1 (EN)
- net at U4.A1 (GPOUT): now also R40.1
- net at U4.B1 (BIN): now also R41.2
- net at U4.B3 (VDD): now also C63.1, C64.1
- net +BATT: now reaches U4.C1 (SRP)
- net +BATT: now also U4.C3 (BAT), C65.1, J5.1 (Pin_1), R42.1
- net at U2.10 (LIIM): now also R37.2
- net at U2.11 (TS): now also J5.2 (Pin_2), R38.2, R39.2, R43.1
- net at U2.19 (SW): now also U2.20 (SW), C58.1, L4.1
- net at U2.21 (BTST): now also C58.2
- net at U2.22 (REGN): now also C57.1, R39.1
- new net: C74.1, C75.1, FB5.1, U15.5 (VCC)
- new net: C73.1, U15.4 (Y)
- new net: C68.1, C69.1, C70.1, L6.1, R44.1, R45.1, U5.A1 (FB)
- new net: L5.1, U5.B2 (SW)
- new net: L6.2, R46.2, R47.2
- new net: L5.2, R44.2, R45.2
- new net: Q5.6 (C1), Q6.1 (G), R49.1
- new net: C73.2, L7.1
- new net DRV_A: R51.2, U15.2 (A)
- new net TX_EN: D12.3 (COM), R50.1
- new net ~{DRV_OE}: C72.2, D12.1 (A), R50.2, U15.1 (~{OE})
Other:
- note added: "If using thermistor, remove R43"
- moved on the sheet: C22, C23, C24, C25, C54, C55, C56, J2, J3, J4, JP1, Q4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

Commit message: fixed stuff
Parts:
- removed FLT1: ~, LFL182G45TC1A108, symbol linea:LFL182G45TC1A108
- added FB4: 100R, Inductor_SMD:L_0603_1608Metric, symbol Device:FerriteBead_Small
- added FL1: ~, LFL182G45TC1A108:FILTET-SMD_0603-6P-L1.6-W0.8-P0.50_LFL182G45TC1A108, symbol LFL182G45TC1A108:LFL182G45TC1A108
- added J6, J7: Conn_01x03_Pin, symbol Connector:Conn_01x03_Pin
- U1: value STM32WB55RGVx -> STM32WB55RGV6TR
- renumbered U8 to U10
Connections:
- net GNDS is gone; now on net GND: JP1.1 (A)
- net TIM8_CH1 is gone; now on net TIM1_CH1: C22.2
- net ~{TIM8_CH1} is gone; now on net ~{TIM1_CH1}: C24.2
- net ~{TIM8_CH3} is gone; now on net ~{TIM1_CH3}: C25.2
- net +3.3V: now also SW2.2, FB4.2; no longer C7.1, C8.1, U1.14 (VDDA)
- net +5V: now also FB5.2
- net +BATT: now also J7.1 (Pin_1)
- net ADC1_IN3: now also U1.11 (PC2)
- net BOOT: now also R10.2
- net BUTTON: now also R11.2
- net EXCITER: now also U1.66 (PB6)
- net GND: now also SW1.2, SW3.2, FL1.2 (GND), FL1.5 (GND), J6.3 (Pin_3), J7.3 (Pin_3)
- net I2C_SCL: now also U1.6 (PB8); no longer U1.24 (PA9)
- net I2C_SDA: now also U1.7 (PB9); no longer U1.51 (PA10)
- net RESET: now also R9.2
- net S0: now also U1.58 (PC10)
- net S1: now also U1.57 (PA15)
- net S2: now also U1.56 (PA14)
- net TIM2_CH1: now also U1.15 (PA0)
- net TIM2_CH2: now also U1.16 (PA1)
- net TX_EN: now also U1.46 (PB12)
- net VBUS: no longer FB5.2
- net ~{E0}: now also U1.65 (PB5)
- net ~{E1}: now also U1.64 (PB4)
- net ~{E2}: now also U1.63 (PB3)
- net ~{E3}: now also U1.62 (PD1)
- net ~{E4}: now also U1.61 (PD0)
- net ~{E5}: now also U1.60 (PC12)
- net TIM2_CH3: now reaches U1.17 (PA2)
- net ~{TIM1_CH1}: now reaches U1.22 (PA7)
- net TIM1_CH1: now reaches U1.23 (PA8)
- net ~{TIM1_CH3}: now reaches U1.49 (PB15)
- net RX: now reaches U1.67 (PB7)
- net RX: now also J6.2 (Pin_2)
- net at J5.2 (Pin_2), R38.2, R39.2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: now also J7.2 (Pin_2)
- net at C17.1, L2.2: now also FL1.1 (IN)
- net at C18.1, L3.1: now also FL1.3 (OUT)
- net TIM8_CH3 renamed TIM1_CH3
- net TIM1_CH3: now also U1.51 (PA10)
- new net TX: J6.1 (Pin_1), U1.24 (PA9)
- new net VDDA: C7.1, C8.1, FB4.1, U1.14 (VDDA)
- no-connect marks 34 -> 58
Other:
- title: (none) -> Linea Main Board
- moved on the sheet: C8, R10, R11, R9, SW1, SW2, SW3

Commit message: update footprints
Parts:
- removed U15: SN74LV1T125DCK, Package_TO_SOT_SMD:SOT-353_SC-70-5, symbol Logic_LevelTranslator:SN74LV1T125DCK
- added U13: SN74LV1T125DCKR, linea:SC-70-5_L2.1-W1.3-P0.65-LS2.1-TL, symbol linea:SN74LV1T125DCKR
- C1, C10, C11, C12, C13, C14, C15, C16, C17, C18, C19, C2, C20, C21, C3, C4, C5, C55, C56, C57, C58, C59, C6, C60, C61, C62, C63, C64, C65, C66, C67, C68, C69, C7, C70, C71, C8, C9: footprint (none) -> Capacitor_SMD:C_0402_1005Metric
- C22, C23, C24, C25: footprint Capacitor_SMD:C_0402_1005Metric_Pad0.74x0.62mm_HandSolder -> Capacitor_SMD:C_0402_1005Metric
- FL1: footprint LFL182G45TC1A108:FILTET-SMD_0603-6P-L1.6-W0.8-P0.50_LFL182G45TC1A108 -> linea:FILTET-SMD_0603-6P-L1.6-W0.8-P0.50_LFL182G45TC1A108
- J1: footprint (none) -> USB-C-Power-tester:TYPE-C-31-M-17
- J5: footprint (none) -> Connector_JST:JST_EH_S3B-EH_1x03_P2.50mm_Horizontal
- J6, J7: footprint (none) -> PCM_4ms_Connector:Pins_1x03_2.54mm_TH
- L1, L2, L3, L4, L5, L6: footprint (none) -> Inductor_SMD:L_0603_1608Metric
- Q4: footprint DMN313DLT-7:SOT-523-3_L1.6-W0.8-P1.00-LS1.6-BR -> linea:SOT-523-3_L1.6-W0.8-P1.00-LS1.6-BR
- Q5: footprint MMDT2907A-7-F:SOT-363_L2.0-W1.3-P0.65-LS2.1-BL -> linea:SOT-363_L2.0-W1.3-P0.65-LS2.1-BL
- Q6: footprint DMP1045U-7:SOT-23-3_L2.9-W1.3-P1.90-LS2.4-BR -> linea:SOT-23-3_L2.9-W1.3-P1.90-LS2.4-BR
- R1, R10, R11, R2, R3, R31, R32, R33, R34, R35, R36, R37, R38, R39, R4, R40, R41, R42, R43, R44, R45, R46, R47, R48, R49, R5, R6, R7, R8, R9: footprint (none) -> Resistor_SMD:R_0402_1005Metric
- U2: footprint BQ25896RTWR:QFN-24_L4.0-W4.0-P0.50-TL-EP2.7 -> linea:QFN-24_L4.0-W4.0-P0.50-TL-EP2.7
- U3: footprint RS3221-3.3YF3:SOT-23-3_L2.9-W1.6-P1.90-LS2.8-BR -> linea:SOT-23-3_L2.9-W1.6-P1.90-LS2.8-BR
- U4: footprint BQ27220YZFR:DSBGA-9_L1.7-W1.6-R3-C3-P0.50-BL -> linea:DSBGA-9_L1.7-W1.6-R3-C3-P0.50-BL
- U5: footprint LM3281YFQR:DSBGA-6_L1.4-W1.1-R3-C2-P0.40-BL -> linea:DSBGA-6_L1.4-W1.1-R3-C2-P0.40-BL
Connections:
- net DRV_A: now also U13.2 (A)
- net VSSA: now also U13.3 (GND)
- net ~{DRV_OE}: now also U13.1 (#OE)
- net at C74.1, C75.1, FB5.1: now also U13.5 (VCC)
- net at C73.1: now also U13.4 (Y)
Other:
- moved on the sheet: C73, L7

Commit message: added more stuff
Parts:
- added X1: XOS32032000LT00351005, linea:OSC-SMD_4P-L3.2-W2.5-BL, symbol linea:XOS32032000LT00351005
- SW1, SW2: footprint (none) -> Button_Switch_SMD:SW_SPST_CK_RS282G05A3
Other:
- moved on the sheet: C10, C15, C9, L1
Changed lines of the file:
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@@
 	)
 	(junction
-		(at 181.61 58.42)
+		(at 191.77 58.42)
 		(diameter 0)
 		(color 0 0 0 0)
@@
 	)
 	(junction
-		(at 196.85 55.88)
+		(at 207.01 55.88)
 		(diameter 0)
 		(color 0 0 0 0)
@@
 	)
 	(junction
-		(at 181.61 66.04)
+		(at 191.77 66.04)
 		(diameter 0)
 		(color 0 0 0 0)
@@
 	)
 	(junction
-		(at 185.42 66.04)
+		(at 195.58 66.04)
 		(diameter 0)
 		(color 0 0 0 0)
@@
 	(wire
 		(pts
-			(xy 181.61 66.04) (xy 179.07 66.04)
+			(xy 191.77 66.04) (xy 189.23 66.04)
 		)
 		(stroke
@@
 	(wire
 		(pts
-			(xy 181.61 66.04) (xy 185.42 66.04)
+			(xy 191.77 66.04) (xy 195.58 66.04)
 		)
 		(stroke
@@
 	(wire
 		(pts
-			(xy 181.61 58.42) (xy 189.23 58.42)
+			(xy 191.77 58.42) (xy 199.39 58.42)
 		)
 		(stroke
@@
 	(wire
 		(pts
-			(xy 199.39 55.88) (xy 199.39 71.12)
+			(xy 209.55 55.88) (xy 209.55 71.12)
 		)
 		(stroke
@@
 	(wire
 		(pts
-			(xy 196.85 63.5) (xy 196.85 64.77)
+			(xy 207.01 63.5) (xy 207.01 64.77)
+		)
+		(stroke
+			(width 0)
+			(type default)
+		)
+	)
+	(wire
+		(pts
+			(xy 189.23 64.77) (xy 179.07 64.77)
 		)
 		(stroke
@@
 	(wire
 		(pts
-			(xy 162.56 58.42) (xy 181.61 58.42)
+			(xy 162.56 58.42) (xy 191.77 58.42)
 		)
 		(stroke
@@
 	(wire
 		(pts
-			(xy 185.42 66.04) (xy 189.23 66.04)
+			(xy 195.58 66.04) (xy 199.39 66.04)
 		)
 		(stroke
@@
 	(wire
 		(pts
-			(xy 162.56 71.12) (xy 199.39 71.12)
+			(xy 162.56 71.12) (xy 209.55 71.12)
 		)
 		(stroke
@@
 	(wire
 		(pts
-			(xy 179.07 66.04) (xy 179.07 64.77)
+			(xy 189.23 66.04) (xy 189.23 64.77)
 		)
 		(stroke
@@
 	(wire
 		(pts
-			(xy 196.85 55.88) (xy 199.39 55.88)
+			(xy 207.01 55.88) (xy 209.55 55.88)
 		)
 		(stroke
@@
 	(wire
 		(pts
-			(xy 162.56 55.88) (xy 189.23 55.88)
+			(xy 162.56 55.88) (xy 199.39 55.88)
 		)
 		(stroke
@@
 	(symbol
 		(lib_id "Device:C")
-		(at 196.85 59.69 0)
+		(at 207.01 59.69 0)
 		(unit 1)
 		(exclude_from_sim no)
@@
 		(dnp no)
 		(property "Reference" "C15"
-			(at 197.358 57.658 0)
+			(at 207.518 57.658 0)
 			(effects
 				(font
@@
 		)
 		(property "Value" "4.7uF"
-			(at 197.358 62.23 0)
+			(at 207.518 62.23 0)
 			(effects
 				(font
@@
 		)
 		(property "Footprint" "Capacitor_SMD:C_0402_1005Metric"
-			(at 197.8152 63.5 0)
+			(at 207.9752 63.5 0)
 			(effects
 				(font
@@
 		)
 		(property "Datasheet" "~"
-			(at 196.85 59.69 0)
+			(at 207.01 59.69 0)
 			(effects
 				(font
@@
 		)
 		(property "Description" "Unpolarized capacitor"
-			(at 196.85 59.69 0)
+			(at 207.01 59.69 0)
 			(effects
 				(font
@@
 			)
 		)
-		(property "Footprint" ""
+		(property "Footprint" "Button_Switch_SMD:SW_SPST_CK_RS282G05A3"
 			(at 262.89 143.51 0)
 			(effects
@@
 			)
 		)
-		(property "Footprint" ""
+		(property "Footprint" "Button_Switch_SMD:SW_SPST_CK_RS282G05A3"
 			(at 262.89 128.27 0)
 			(effects
@@
 	(symbol
 		(lib_id "Device:L")
-		(at 193.04 55.88 90)
+		(at 203.2 55.88 90)
 		(unit 1)
 		(exclude_from_sim no)
@@
 		(dnp no)
 		(property "Reference" "L1"
-			(at 190.754 53.848 90)
+			(at 200.914 53.848 90)
 			(effects
 				(font
@@
 		)
 		(property "Value" "10uH"
-			(at 195.326 53.848 90)
+			(at 205.486 53.848 90)
 			(effects
 				(font
@@
 		)
 		(property "Footprint" "Inductor_SMD:L_0603_1608Metric"
-			(at 193.04 55.88 0)
+			(at 203.2 55.88 0)
 			(effects
 				(font
@@
 		)
 		(property "Datasheet" "~"
-			(at 193.04 55.88 0)
+			(at 203.2 55.88 0)
 			(effects
 				(font
@@
 		)
 		(property "Description" "Inductor"
-			(at 193.04 55.88 0)
+			(at 203.2 55.88 0)
 			(effects
 				(font
@@
 	)
 	(symbol
+		(lib_id "linea:XOS32032000LT00351005")
+		(at 196.85 102.87 0)
+		(unit 1)
+		(exclude_from_sim no)
+		(in_bom yes)
+		(on_board yes)
+		(dnp no)
+		(fields_autoplaced yes)
+		(property "Reference" "X1"
+			(at 196.85 93.98 0)
+			(effects
+				(font
+					(size 1.27 1.27)
+				)
+			)
+		)
+		(property "Value" "XOS32032000LT00351005"
+			(at 196.85 96.52 0)
+			(effects
+				(font
+					(size 1.27 1.27)
+				)
+			)
+		)
+		(property "Footprint" "linea:OSC-SMD_4P-L3.2-W2.5-BL"
+			(at 196.85 111.76 0)
+			(effects
+				(font
+					(size 1.27 1.27)
+				)
+				(hide yes)
+			)
+		)
+		(property "Datasheet" ""
+			(at 196.85 102.87 0)
+			(effects
+				(font
+					(size 1.27 1.27)
+				)
+				(hide yes)
+			)
+		)
+		(property "Description" ""
+			(at 196.85 102.87 0)
+			(effects
+				(font
+					(size 1.27 1.27)
+				)
+				(hide yes)
+			)
+		)
+		(property "LCSC Part" "C37635419"
+			(at 196.85 114.3 0)
+			(effects
+				(font
+					(size 1.27 1.27)
+				)
+				(hide yes)
+			)
+		)
+		(pin "3"
+		)
+		(pin "4"
+		)
+		(pin "2"
+		)
+		(pin "1"
+		)
+		(instances
+			(project ""
+				(path "/f5ca596a-3f37-4a80-af8e-71fb2890766f"
+					(reference "X1")
+					(unit 1)
+				)
+			)
+		)
+	)
+	(symbol
 		(lib_id "Device:C")
 		(at 133.35 22.86 0)
@@
 	(symbol
 		(lib_id "power:GND")
-		(at 196.85 64.77 0)
+		(at 207.01 64.77 0)
 		(unit 1)
 		(exclude_from_sim no)
@@
 		(dnp no)
 		(property "Reference" "#PWR08"
-			(at 196.85 71.12 0)
+			(at 207.01 71.12 0)
 			(effects
 				(font
@@
 		)
 		(property "Value" "GND"
-			(at 196.85 68.834 0)
+			(at 207.01 68.834 0)
 			(effects
 				(font
@@
 		)
 		(property "Footprint" ""
-			(at 196.85 64.77 0)
+			(at 207.01 64.77 0)
 			(effects
 				(font
@@
 		)
 		(property "Datasheet" ""
-			(at 196.85 64.77 0)
+			(at 207.01 64.77 0)
 			(effects
 				(font
@@
 		)
 		(property "Description" "Power symbol creates a global label with name \"GND\" , ground"
-			(at 196.85 64.77 0)
+			(at 207.01 64.77 0)
 			(effects
 				(font
@@
 	(symbol
 		(lib_id "Device:C")
-		(at 189.23 62.23 0)
+		(at 199.39 62.23 0)
 		(unit 1)
 		(exclude_from_sim no)
@@
 		(dnp no)
 		(property "Reference" "C10"
-			(at 189.738 60.198 0)
+			(at 199.898 60.198 0)
 			(effects
 				(font
@@
 		)
 		(property "Value" "100nF"
-			(at 189.738 64.77 0)
+			(at 199.898 64.77 0)
 			(effects
 				(font
@@
 		)
 		(property "Footprint" "Capacitor_SMD:C_0402_1005Metric"
-			(at 190.1952 66.04 0)
+			(at 200.3552 66.04 0)
 			(effects
 				(font
@@
 		)
 		(property "Datasheet" "~"
-			(at 189.23 62.23 0)
+			(at 199.39 62.23 0)
 			(effects
 				(font
@@
 		)
 		(property "Description" "Unpolarized capacitor"
-			(at 189.23 62.23 0)
+			(at 199.39 62.23 0)
 			(effects
 				(font
@@
 	(symbol
 		(lib_id "power:GND")
-		(at 185.42 66.04 0)
+		(at 195.58 66.04 0)
 		(unit 1)
 		(exclude_from_sim no)
@@
 		(dnp no)
 		(property "Reference" "#PWR07"
-			(at 185.42 72.39 0)
+			(at 195.58 72.39 0)
 			(effects
 				(font
@@
 		)
 		(property "Value" "GND"
-			(at 185.42 69.85 0)
+			(at 195.58 69.85 0)
 			(effects
 				(font
@@
 		)
 		(property "Footprint" ""
-			(at 185.42 66.04 0)
+			(at 195.58 66.04 0)
 			(effects
 				(font
@@
 		)
 		(property "Datasheet" ""
-			(at 185.42 66.04 0)
+			(at 195.58 66.04 0)
 			(effects
 				(font
@@
 		)
 		(property "Description" "Power symbol creates a global label with name \"GND\" , ground"
-			(at 185.42 66.04 0)
+			(at 195.58 66.04 0)
 			(effects
 				(font
@@
 	(symbol
 		(lib_id "Device:C")
-		(at 181.61 62.23 0)
+		(at 191.77 62.23 0)
 		(unit 1)
 		(exclude_from_sim no)
@@
 		(dnp no)
 		(property "Reference" "C9"
-			(at 182.118 60.198 0)
+			(at 192.278 60.198 0)
 			(effects
 				(font
@@
 		)
 		(property "Value" "1uF"
-			(at 182.118 64.77 0)
+			(at 192.278 64.77 0)
 			(effects
 				(font
@@
 		)
 		(property "Footprint" "Capacitor_SMD:C_0402_1005Metric"
-			(at 182.5752 66.04 0)
+			(at 192.7352 66.04 0)
 			(effects
 				(font
@@
 		)
 		(property "Datasheet" "~"
-			(at 181.61 62.23 0)
+			(at 191.77 62.23 0)
 			(effects
 				(font
@@
 		)
 		(property "Description" "Unpolarized capacitor"
-			(at 181.61 62.23 0)
+			(at 191.77 62.23 0)
 			(effects
 				(font
