File: hardware/board/board.kicad_sch (KiCad schematic)
At the start: 135 parts, among them J1 USB_C_Receptacle, J2 Conn_01x26_MountingPin, J3 Conn_01x26_MountingPin, J4 Conn_01x26_MountingPin, J5 Conn_01x03, J6 Conn_01x03_Pin, J7 Conn_01x03_Pin, SW1 SW_Push, SW2 SW_Push, SW3 SW_Push, U1 STM32WB55RGV6TR, U10 74HC4051, U11 74HC4051, U12 74HC4051, U13 SN74LV1T125DCKR, U7 74HC4051, U8 74HC4051, U9 74HC4051, X1 XOS32032000LT00351005, Y1 32MHz, Y2 32.768kHz

Commit message: fnished shcamtic
Parts:
- removed SW3: SW_Push, symbol Switch:SW_Push
- removed X1: XOS32032000LT00351005, linea:OSC-SMD_4P-L3.2-W2.5-BL, symbol linea:XOS32032000LT00351005
- removed Y1: 32MHz, symbol Device:Crystal_GND3
- removed Y2: 32.768kHz, symbol Device:Crystal
- added SW3: SKRTLAE010, linea:KEY-SMD_SKRTLAE010, symbol linea:SKRTLAE010
- added X1: XL7EL89CKI-111YLC-32M, linea:CRYSTAL-SMD_4P-L2.0-W1.6-BL, symbol linea:XL7EL89CKI-111YLC-32M
- added X2: FC-12M32.768KHZ7PF20PPM, linea:FC-12M_L2.0-W1.2, symbol linea:FC-12M32.768KHZ7PF20PPM
- J1: footprint USB-C-Power-tester:TYPE-C-31-M-17 -> Connector_USB:USB_C_Receptacle_Amphenol_12401548E4-2A
Connections:
- net BUTTON: now also SW3.2
- net GND: now also J2.13 (Pin_13), J2.18 (Pin_18), J2.23 (Pin_23), J2.3 (Pin_3), J2.8 (Pin_8), J3.13 (Pin_13), J3.18 (Pin_18), J3.23 (Pin_23), J3.3 (Pin_3), J3.8 (Pin_8), J4.13 (Pin_13), J4.18 (Pin_18), J4.23 (Pin_23), J4.3 (Pin_3), J4.8 (Pin_8), SW3.1, SW3.3, SW3.4, SW3.5, X1.2 (GND), X1.4 (GND); no longer J2.14 (Pin_14), J2.19 (Pin_19), J2.24 (Pin_24), J2.4 (Pin_4), J2.9 (Pin_9), J3.14 (Pin_14), J3.19 (Pin_19), J3.24 (Pin_24), J3.4 (Pin_4), J3.9 (Pin_9), J4.14 (Pin_14), J4.19 (Pin_19), J4.24 (Pin_24), J4.4 (Pin_4), J4.9 (Pin_9)
- net X0: now also J4.1 (Pin_1); no longer J4.26 (Pin_26)
- net X1: now also J4.2 (Pin_2); no longer J4.25 (Pin_25)
- net X10: now also J4.14 (Pin_14); no longer J4.13 (Pin_13)
- net X11: now also J4.15 (Pin_15); no longer J4.12 (Pin_12)
- net X12: now also J4.16 (Pin_16); no longer J4.11 (Pin_11)
- net X13: now also J4.17 (Pin_17); no longer J4.10 (Pin_10)
- net X14: now also J4.19 (Pin_19); no longer J4.8 (Pin_8)
- net X15: now also J4.20 (Pin_20); no longer J4.7 (Pin_7)
- net X16: now also J4.21 (Pin_21); no longer J4.6 (Pin_6)
- net X17: now also J4.22 (Pin_22); no longer J4.5 (Pin_5)
- net X18: now also J4.24 (Pin_24); no longer J4.3 (Pin_3)
- net X19: now also J4.25 (Pin_25); no longer J4.2 (Pin_2)
- net X2: now also J4.4 (Pin_4); no longer J4.23 (Pin_23)
- net X20: now also J3.1 (Pin_1); no longer J3.26 (Pin_26)
- net X21: now also J3.2 (Pin_2); no longer J3.25 (Pin_25)
- net X22: now also J3.4 (Pin_4); no longer J3.23 (Pin_23)
- net X23: now also J3.5 (Pin_5); no longer J3.22 (Pin_22)
- net X24: now also J3.6 (Pin_6); no longer J3.21 (Pin_21)
- net X25: now also J3.7 (Pin_7); no longer J3.20 (Pin_20)
- net X26: now also J3.9 (Pin_9); no longer J3.18 (Pin_18)
- net X27: now also J3.10 (Pin_10); no longer J3.17 (Pin_17)
- net X3: now also J4.5 (Pin_5); no longer J4.22 (Pin_22)
- net X4: now also J4.6 (Pin_6); no longer J4.21 (Pin_21)
- net X5: now also J4.7 (Pin_7); no longer J4.20 (Pin_20)
- net X6: now also J4.9 (Pin_9); no longer J4.18 (Pin_18)
- net X7: now also J4.10 (Pin_10); no longer J4.17 (Pin_17)
- net X8: now also J4.11 (Pin_11); no longer J4.16 (Pin_16)
- net X9: now also J4.12 (Pin_12); no longer J4.15 (Pin_15)
- net Y0: now also J2.1 (Pin_1); no longer J2.26 (Pin_26)
- net Y1: now also J2.2 (Pin_2); no longer J2.25 (Pin_25)
- net Y10: now also J2.14 (Pin_14); no longer J2.13 (Pin_13)
- net Y11: now also J2.15 (Pin_15); no longer J2.12 (Pin_12)
- net Y12: now also J2.16 (Pin_16); no longer J2.11 (Pin_11)
- net Y13: now also J2.17 (Pin_17); no longer J2.10 (Pin_10)
- net Y14: now also J2.19 (Pin_19); no longer J2.8 (Pin_8)
- net Y15: now also J2.20 (Pin_20); no longer J2.7 (Pin_7)
- net Y16: now also J2.21 (Pin_21); no longer J2.6 (Pin_6)
- net Y17: now also J2.22 (Pin_22); no longer J2.5 (Pin_5)
- net Y2: now also J2.4 (Pin_4); no longer J2.23 (Pin_23)
- net Y3: now also J2.5 (Pin_5); no longer J2.22 (Pin_22)
- net Y4: now also J2.6 (Pin_6); no longer J2.21 (Pin_21)
- net Y5: now also J2.7 (Pin_7); no longer J2.20 (Pin_20)
- net Y6: now also J2.9 (Pin_9); no longer J2.18 (Pin_18)
- net Y7: now also J2.10 (Pin_10); no longer J2.17 (Pin_17)
- net Y8: now also J2.11 (Pin_11); no longer J2.16 (Pin_16)
- net Y9: now also J2.12 (Pin_12); no longer J2.15 (Pin_15)
- net at C20.1, U1.4 (PC15): now also X2.1 (OSC1)
- net at C21.1, U1.3 (PC14): now also X2.2 (OSC2)
- net at U1.34 (OSC_OUT): now also X1.1
- net at U1.35 (OSC_IN): now also X1.3
Other:
- moved on the sheet: C20

Commit message: added touches
Parts:
- U10, U11, U12, U7, U8, U9: footprint Package_DFN_QFN:DHVQFN-16-1EP_2.5x3.5mm_P0.5mm_EP1x2mm -> Package_SO:TSSOP-16_4.4x5mm_P0.65mm
Connections:
- net GND: now also J2.14 (Pin_14), J2.19 (Pin_19), J2.24 (Pin_24), J2.4 (Pin_4), J2.9 (Pin_9); no longer J2.13 (Pin_13), J2.18 (Pin_18), J2.23 (Pin_23), J2.3 (Pin_3), J2.8 (Pin_8)
- net X0: now also U7.14 (A1); no longer U7.13 (A0)
- net X1: now also U7.15 (A2); no longer U7.14 (A1)
- net X10: now also U8.1 (A4); no longer U8.15 (A2)
- net X11: now also U8.2 (A6); no longer U8.12 (A3)
- net X12: now also U8.4 (A7); no longer U8.1 (A4)
- net X14: now also U9.12 (A3); no longer U8.2 (A6)
- net X15: now also U9.13 (A0); no longer U8.4 (A7)
- net X16: now also U9.14 (A1); no longer U9.13 (A0)
- net X17: now also U9.15 (A2); no longer U9.14 (A1)
- net X18: now also U9.1 (A4); no longer U9.15 (A2)
- net X19: now also U9.2 (A6); no longer U9.12 (A3)
- net X2: now also U7.1 (A4); no longer U7.15 (A2)
- net X20: now also U9.4 (A7); no longer U9.1 (A4)
- net X22: now also U10.12 (A3); no longer U9.2 (A6)
- net X23: now also U10.13 (A0); no longer U9.4 (A7)
- net X24: now also U10.14 (A1); no longer U10.13 (A0)
- net X25: now also U10.15 (A2); no longer U10.14 (A1)
- net X26: now also U10.1 (A4); no longer U10.15 (A2)
- net X27: now also U10.2 (A6); no longer U10.12 (A3)
- net X3: now also U7.2 (A6); no longer U7.12 (A3)
- net X4: now also U7.4 (A7); no longer U7.1 (A4)
- net X6: now also U8.12 (A3); no longer U7.2 (A6)
- net X7: now also U8.13 (A0); no longer U7.4 (A7)
- net X8: now also U8.14 (A1); no longer U8.13 (A0)
- net X9: now also U8.15 (A2); no longer U8.14 (A1)
- net Y0: now also J2.26 (Pin_26), U11.15 (A2); no longer J2.1 (Pin_1), U10.1 (A4)
- net Y1: now also J2.25 (Pin_25), U11.14 (A1); no longer J2.2 (Pin_2), U10.5 (A5)
- net Y10: now also J2.13 (Pin_13), U12.14 (A1); no longer J2.14 (Pin_14), U11.2 (A6)
- net Y11: now also J2.12 (Pin_12), U12.15 (A2); no longer J2.15 (Pin_15), U11.4 (A7)
- net Y12: now also J2.11 (Pin_11), U12.1 (A4); no longer J2.16 (Pin_16), U12.13 (A0)
- net Y13: now also J2.10 (Pin_10), U12.2 (A6); no longer J2.17 (Pin_17), U12.14 (A1)
- net Y14: now also J2.8 (Pin_8), U12.4 (A7); no longer J2.19 (Pin_19), U12.15 (A2)
- net Y15: now also J2.7 (Pin_7), U12.5 (A5); no longer J2.20 (Pin_20), U12.12 (A3)
- net Y16: now also J2.6 (Pin_6), U7.12 (A3); no longer J2.21 (Pin_21), U12.1 (A4)
- net Y17: now also J2.5 (Pin_5), U7.13 (A0); no longer J2.22 (Pin_22), U12.5 (A5)
- net Y2: now also J2.23 (Pin_23), U11.13 (A0); no longer J2.4 (Pin_4), U10.2 (A6)
- net Y3: now also J2.22 (Pin_22), U11.12 (A3); no longer J2.5 (Pin_5), U10.4 (A7)
- net Y4: now also J2.21 (Pin_21), U11.5 (A5); no longer J2.6 (Pin_6), U11.13 (A0)
- net Y5: now also J2.20 (Pin_20), U11.4 (A7); no longer J2.7 (Pin_7), U11.14 (A1)
- net Y6: now also J2.18 (Pin_18), U11.2 (A6); no longer J2.9 (Pin_9), U11.15 (A2)
- net Y7: now also J2.17 (Pin_17), U11.1 (A4); no longer J2.10 (Pin_10), U11.12 (A3)
- net Y8: now also J2.16 (Pin_16), U12.12 (A3); no longer J2.11 (Pin_11), U11.1 (A4)
- net Y9: now also J2.15 (Pin_15), U12.13 (A0); no longer J2.12 (Pin_12), U11.5 (A5)

Commit message: pcb power start
Parts:
- removed D1, D2: PESD15VL1BA, PCM_Diode_SMD_AKL:D_SOD-323_TVS, symbol PCM_Diode_TVS_AKL:PESD15VL1BA
- removed J1: USB_C_Receptacle, Connector_USB:USB_C_Receptacle_Amphenol_12401548E4-2A, symbol Connector:USB_C_Receptacle
- removed R3, R4: 22, Resistor_SMD:R_0402_1005Metric, symbol Device:R
- added L8: EXC14CE900U, linea:FILTER-SMD_4P-L0.9-W0.7-P0.50-BL, symbol linea:EXC14CE900U
- added U14: USBLC6-2P6, Package_TO_SOT_SMD:SOT-666, symbol Power_Protection:USBLC6-2P6
- added USB1: TYPE-C 16PIN 2MD(073), linea:USB-C-SMD_TYPE-C-6PIN-2MD-073, symbol linea:TYPE-C16PIN2MD(073)
Connections:
- net GND: now also J3.14 (Pin_14), J3.19 (Pin_19), J3.24 (Pin_24), J3.4 (Pin_4), J3.9 (Pin_9), J4.14 (Pin_14), J4.19 (Pin_19), J4.24 (Pin_24), J4.4 (Pin_4), J4.9 (Pin_9), U14.2 (GND), USB1.1 (GND), USB1.12 (GND), USB1.13 (SHELL), USB1.14 (SHELL); no longer J3.13 (Pin_13), J3.18 (Pin_18), J3.23 (Pin_23), J3.3 (Pin_3), J3.8 (Pin_8), J4.13 (Pin_13), J4.18 (Pin_18), J4.23 (Pin_23), J4.3 (Pin_3), J4.8 (Pin_8)
- net VBUS: now also U14.5 (VBUS), USB1.11 (VBUS), USB1.2 (VBUS)
- net X0: now also J3.26 (Pin_26); no longer J4.1 (Pin_1)
- net X1: now also J3.25 (Pin_25); no longer J4.2 (Pin_2)
- net X10: now also J3.13 (Pin_13); no longer J4.14 (Pin_14)
- net X11: now also J3.12 (Pin_12); no longer J4.15 (Pin_15)
- net X12: now also J3.11 (Pin_11); no longer J4.16 (Pin_16)
- net X13: now also J3.10 (Pin_10); no longer J4.17 (Pin_17)
- net X14: now also J3.8 (Pin_8); no longer J4.19 (Pin_19)
- net X15: now also J3.7 (Pin_7); no longer J4.20 (Pin_20)
- net X16: now also J3.6 (Pin_6); no longer J4.21 (Pin_21)
- net X17: now also J3.5 (Pin_5); no longer J4.22 (Pin_22)
- net X18: now also J3.3 (Pin_3); no longer J4.24 (Pin_24)
- net X19: now also J3.2 (Pin_2); no longer J4.25 (Pin_25)
- net X2: now also J3.23 (Pin_23); no longer J4.4 (Pin_4)
- net X20: now also J4.26 (Pin_26); no longer J3.1 (Pin_1)
- net X21: now also J4.25 (Pin_25); no longer J3.2 (Pin_2)
- net X22: now also J4.23 (Pin_23); no longer J3.4 (Pin_4)
- net X23: now also J4.22 (Pin_22); no longer J3.5 (Pin_5)
- net X24: now also J4.21 (Pin_21); no longer J3.6 (Pin_6)
- net X25: now also J4.20 (Pin_20); no longer J3.7 (Pin_7)
- net X26: now also J4.18 (Pin_18); no longer J3.9 (Pin_9)
- net X27: now also J4.17 (Pin_17); no longer J3.10 (Pin_10)
- net X3: now also J3.22 (Pin_22); no longer J4.5 (Pin_5)
- net X4: now also J3.21 (Pin_21); no longer J4.6 (Pin_6)
- net X5: now also J3.20 (Pin_20); no longer J4.7 (Pin_7)
- net X6: now also J3.18 (Pin_18); no longer J4.9 (Pin_9)
- net X7: now also J3.17 (Pin_17); no longer J4.10 (Pin_10)
- net X8: now also J3.16 (Pin_16); no longer J4.11 (Pin_11)
- net X9: now also J3.15 (Pin_15); no longer J4.12 (Pin_12)
- net Y0: now also U11.12 (A3); no longer U11.15 (A2)
- net Y1: now also U11.13 (A0); no longer U11.14 (A1)
- net Y2: now also U11.14 (A1); no longer U11.13 (A0)
- net Y3: now also U11.15 (A2); no longer U11.12 (A3)
- net Y4: now also U11.1 (A4); no longer U11.5 (A5)
- net Y5: now also U11.2 (A6); no longer U11.4 (A7)
- net Y6: now also U11.4 (A7); no longer U11.2 (A6)
- net Y7: now also U11.5 (A5); no longer U11.1 (A4)
- net at U1.52 (PA11): now also L8.2
- net at U1.53 (PA12): now also L8.1
- net at R2.1: now also USB1.10 (CC2)
- net at R1.1: now also USB1.4 (CC1)
- new net: L8.3, U14.1 (I/O1), U14.6 (I/O1), USB1.6 (DP1), USB1.8 (DP2)
- new net: L8.4, U14.3 (I/O2), U14.4 (I/O2), USB1.5 (DN2), USB1.7 (DN1)
- no-connect marks 58 -> 48
Other:
- moved on the sheet: R1, R2
