File: hardware/board/board.kicad_sch (KiCad schematic)
At the start: 132 parts, among them J2 Conn_01x26_MountingPin, J3 Conn_01x26_MountingPin, J4 Conn_01x26_MountingPin, J5 Conn_01x03, J6 Conn_01x03_Pin, J7 Conn_01x03_Pin, SW1 SW_Push, SW2 SW_Push, SW3 SKRTLAE010, U1 STM32WB55RGV6TR, U10 74HC4051, U11 74HC4051, U12 74HC4051, U13 SN74LV1T125DCKR, U14 USBLC6-2P6, U7 74HC4051, U8 74HC4051, U9 74HC4051, X1 XL7EL89CKI-111YLC-32M, X2 FC-12M32.768KHZ7PF20PPM

Commit message: bunch o f stuff
Parts:
- removed AE1: 1001312, symbol Device:Antenna
- removed C16: 0.8pF, Capacitor_SMD:C_0402_1005Metric, symbol Device:C
- removed C17: 0.3pF, Capacitor_SMD:C_0402_1005Metric, symbol Device:C
- removed C18: 1.5pF, Capacitor_SMD:C_0402_1005Metric, symbol Device:C
- removed C19: DNP, Capacitor_SMD:C_0402_1005Metric, symbol Device:C
- removed C44, C45, C46, C47: 100nF, Capacitor_SMD:C_0402_1005Metric, symbol Device:C_Small
- removed FL1: ~, linea:FILTET-SMD_0603-6P-L1.6-W0.8-P0.50_LFL182G45TC1A108, symbol LFL182G45TC1A108:LFL182G45TC1A108
- removed J6, J7: Conn_01x03_Pin, PCM_4ms_Connector:Pins_1x03_2.54mm_TH, symbol Connector:Conn_01x03_Pin
- removed L2: 2.7nH, Inductor_SMD:L_0603_1608Metric, symbol Device:L
- removed L3: 3nH, Inductor_SMD:L_0603_1608Metric, symbol Device:L
- removed R5: 0, Resistor_SMD:R_0402_1005Metric, symbol Device:R
- removed R6, R7, R8: DNP, Resistor_SMD:R_0402_1005Metric, symbol Device:R
- added AE1: 2450AT18A100E, linea:ANT-SMD_L3.2-W1.6, symbol linea:2450AT18A100E
- added C44: 10uF, Capacitor_SMD:C_0402_1005Metric, symbol Device:C
- added C45: 22uF, Capacitor_SMD:C_0402_1005Metric, symbol Device:C
- added D1: 1N4148WT, Diode_SMD:D_SOD-523, symbol Diode:1N4148WT
- added FL2: MLPF-WB55-01E3, linea:FILTER-SMD_6P-L1.6-W1.0-P0.50-BL, symbol linea:MLPF-WB55-01E3
- added L9: 470nH, Inductor_SMD:L_Murata_DFE201610P, symbol Device:L
- added TP1, TP2, TP3: TestPoint, TestPoint:TestPoint_Pad_1.5x1.5mm, symbol Connector:TestPoint
- added U15: FAN48610BUC50X, linea:WLCSP-9_L1.2-W1.2-R3-C3-P0.40-BL, symbol linea:FAN48610BUC50X
Connections:
- net +3.3V: now also C11.1, C12.1, U1.33 (VDDRF)
- net +5V: now also C48.2, C50.2, C52.2, U10.16 (VCC), U11.16 (VCC), U12.16 (VCC), U7.16 (VCC), U8.16 (VCC), U9.16 (VCC), C45.1, U15.A1 (VOUT), U15.A2 (VOUT); no longer C56.1, Q5.4 (E2), Q6.2 (S), U2.1 (VBUS)
- net +BATT: now also TP1.1
- net GND: now also C44.2, C45.2, FL2.2 (GND4), FL2.4 (GND1), FL2.5 (GND2), FL2.6 (GND3), TP3.1, U15.C1 (PGND), U15.C2 (PGND), U15.C3 (AGND); no longer J2.14 (Pin_14), J2.19 (Pin_19), J2.24 (Pin_24), J2.4 (Pin_4), J2.9 (Pin_9), J3.14 (Pin_14), J3.19 (Pin_19), J3.24 (Pin_24), J3.4 (Pin_4), J3.9 (Pin_9), J4.14 (Pin_14), J4.19 (Pin_19), J4.24 (Pin_24), J4.4 (Pin_4), J4.9 (Pin_9), JP1.1 (A)
- net SYS: now also C44.1, L9.1, U15.A3 (VIN), U15.B3 (EN)
- net VBUS: now also D1.1 (K); no longer C48.2, C50.2, C52.2, Q5.2 (B1), Q5.3 (C2), Q5.5 (B2), R48.1, U10.16 (VCC), U11.16 (VCC), U12.16 (VCC), U7.16 (VCC), U8.16 (VCC), U9.16 (VCC)
- net D-: now reaches L8.1, U1.53 (PA12)
- net D+: now reaches L8.2, U1.52 (PA11)
- net at U1.31 (RF1): now also FL2.3 (IN)
- net at J5.2 (Pin_2), R38.2, R39.2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: now also TP2.1
- net RX: no longer names the net of U1.67 (PB7)
- net TX: no longer names the net of U1.24 (PA9)
- new net: D1.2 (A), Q5.2 (B1), Q5.5 (B2)
- new net: Q5.3 (C2), R48.1
- new net: L9.2, U15.B1 (SW), U15.B2 (SW)
- new net: AE1.1 (ANT), FL2.1 (OUT)
- new net GNDS: J2.14 (Pin_14), J2.19 (Pin_19), J2.24 (Pin_24), J2.4 (Pin_4), J2.9 (Pin_9), J3.14 (Pin_14), J3.19 (Pin_19), J3.24 (Pin_24), J3.4 (Pin_4), J3.9 (Pin_9), J4.14 (Pin_14), J4.19 (Pin_19), J4.24 (Pin_24), J4.4 (Pin_4), J4.9 (Pin_9), JP1.1 (A)
- new net USB_5V: C56.1, Q5.4 (E2), Q6.2 (S), U2.1 (VBUS)
- no-connect marks 48 -> 49
Other:
- moved on the sheet: R48

Commit message: finished board
Parts:
- removed C54: 72nF, Capacitor_SMD:C_0402_1005Metric, symbol Device:C_Small
- removed U3: ~, linea:SOT-23-3_L2.9-W1.6-P1.90-LS2.8-BR, symbol RS3221-3.3YF3:RS3221-3.3YF3
- added C16, C19: 3.9nF, Capacitor_SMD:C_0402_1005Metric, symbol Device:C_Small
- added C18: 68nF, Capacitor_SMD:C_0402_1005Metric, symbol Device:C_Small
- added U16: RS3221-3.3YUTDN4, linea:UTDFN-4_L1.0-W1.0-P0.63-BL-EP-1, symbol linea:RS3221-3.3YUTDN4
- C58: value 47uF -> 47nF
- C73: value 72nF -> 68nF
- J2, J3, J4: LCSC (none) -> C262277
- J5: LCSC (none) -> C263754
- L7: LCSC (none) -> C85834
- L9: LCSC (none) -> C882980
- Q4: LCSC (none) -> C155524; Supplier Part C155524 -> (none)
- Q5: LCSC (none) -> C460232; Supplier Part C460232 -> (none)
- Q6: LCSC (none) -> C177033
- SW1, SW2: LCSC (none) -> C318938
- U1: value STM32WB55RGV6TR -> STM32WB55RGV6
- U2: LCSC (none) -> C181475; Supplier Part C181475 -> (none)
- U4: LCSC (none) -> C528617; Supplier Part C528617 -> (none)
- U5: LCSC (none) -> C2070970; Supplier Part C2070970 -> (none)
Connections:
- net ABUS: now also C18.1, C19.1
- net EXCITER: now also C18.2, C19.2
- net GND: now also U16.2 (GND), U16.5 (EP)
- net LDO_3.3V: now also U16.1 (OUT)
- net at C61.1, C62.1, C66.1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: now also U16.3 (EN), U16.4 (IN)
- net at C73.1, U13.4 (Y): now also C16.1
- net at C73.2, L7.1: now also C16.2

Commit message: impdance matching
Other:
- moved on the sheet: R10
Changed lines of the file:
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@@
 	(wire
 		(pts
+			(xy 251.46 151.13) (xy 251.46 148.59)
+		)
+		(stroke
+			(width 0)
+			(type default)
+		)
+	)
+	(wire
+		(pts
 			(xy 162.56 66.04) (xy 166.37 66.04)
 		)
@@
 	(symbol
 		(lib_id "power:GND")
-		(at 251.46 156.21 0)
+		(at 251.46 158.75 0)
 		(unit 1)
 		(exclude_from_sim no)
@@
 		(dnp no)
 		(property "Reference" "#PWR028"
-			(at 251.46 162.56 0)
+			(at 251.46 165.1 0)
 			(effects
 				(font
@@
 		)
 		(property "Value" "GND"
-			(at 251.46 159.766 0)
+			(at 251.46 162.306 0)
 			(effects
 				(font
@@
 		)
 		(property "Footprint" ""
-			(at 251.46 156.21 0)
+			(at 251.46 158.75 0)
 			(effects
 				(font
@@
 		)
 		(property "Datasheet" ""
-			(at 251.46 156.21 0)
+			(at 251.46 158.75 0)
 			(effects
 				(font
@@
 		)
 		(property "Description" "Power symbol creates a global label with name \"GND\" , ground"
-			(at 251.46 156.21 0)
+			(at 251.46 158.75 0)
 			(effects
 				(font
@@
 	(symbol
 		(lib_id "Device:R")
-		(at 251.46 152.4 180)
+		(at 251.46 154.94 180)
 		(unit 1)
 		(exclude_from_sim no)
@@
 		(dnp no)
 		(property "Reference" "R10"
-			(at 252.984 151.13 0)
+			(at 252.984 153.67 0)
 			(effects
 				(font
@@
 		)
 		(property "Value" "10K"
-			(at 252.984 153.67 0)
+			(at 252.984 156.21 0)
 			(effects
 				(font
@@
 		)
 		(property "Footprint" "Resistor_SMD:R_0402_1005Metric"
-			(at 253.238 152.4 90)
+			(at 253.238 154.94 90)
 			(effects
 				(font
@@
 		)
 		(property "Datasheet" "~"
-			(at 251.46 152.4 0)
+			(at 251.46 154.94 0)
 			(effects
 				(font
@@
 		)
 		(property "Description" "Resistor"
-			(at 251.46 152.4 0)
+			(at 251.46 154.94 0)
 			(effects
 				(font

Commit message: esd prtot
Connections:
- net at U14.1 (I/O1), USB1.6 (DP1), USB1.8 (DP2): no longer L8.3, U14.6 (I/O1)
- net at U14.3 (I/O2), USB1.5 (DN2), USB1.7 (DN1): no longer L8.4, U14.4 (I/O2)
- new net: L8.3, U14.6 (I/O1)
- new net: L8.4, U14.4 (I/O2)
Changed lines of the file:
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@@
 	)
 	(junction
-		(at 85.09 78.74)
-		(diameter 0)
-		(color 0 0 0 0)
-	)
-	(junction
 		(at 118.11 228.6)
 		(diameter 0)
@@
 	)
 	(junction
-		(at 71.12 80.01)
-		(diameter 0)
-		(color 0 0 0 0)
-	)
-	(junction
 		(at 388.62 182.88)
 		(diameter 0)
@@
 	)
 	(junction
-		(at 73.66 81.28)
-		(diameter 0)
-		(color 0 0 0 0)
-	)
-	(junction
 		(at 500.38 92.71)
 		(diameter 0)
@@
 	)
 	(junction
-		(at 83.82 81.28)
-		(diameter 0)
-		(color 0 0 0 0)
-	)
-	(junction
 		(at 85.09 312.42)
 		(diameter 0)
@@
 	(wire
 		(pts
-			(xy 77.47 78.74) (xy 77.47 80.01)
-		)
-		(stroke
-			(width 0)
-			(type default)
-		)
-	)
-	(wire
-		(pts
 			(xy 68.58 306.07) (xy 39.37 306.07)
 		)
@@
 	(wire
 		(pts
-			(xy 73.66 81.28) (xy 83.82 81.28)
-		)
-		(stroke
-			(width 0)
-			(type default)
-		)
-	)
-	(wire
-		(pts
 			(xy 229.87 69.85) (xy 229.87 67.31)
 		)
@@
 	(wire
 		(pts
-			(xy 71.12 80.01) (xy 77.47 80.01)
-		)
-		(stroke
-			(width 0)
-			(type default)
-		)
-	)
-	(wire
-		(pts
 			(xy 132.08 43.18) (xy 132.08 34.29)
 		)
@@
 		)
 		(stroke
-			(width 0)
-			(type default)
-		)
-	)
-	(wire
-		(pts
-			(xy 77.47 78.74) (xy 85.09 78.74)
-		)
-		(stroke

Commit message: gerbers
Parts:
- removed R42: 10m, Resistor_SMD:R_0402_1005Metric, symbol Device:R
- added R42: WW25WR010FTL, linea:R2512, symbol linea:WW25WR010FTL
Connections:
- net +BATT: now also R42.2
- net at C61.1, C62.1, C66.1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: now also R42.1
Changed lines of the file:
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@@
 	)
 	(junction
+		(at 149.86 228.6)
+		(diameter 0)
+		(color 0 0 0 0)
+	)
+	(junction
 		(at 195.58 182.88)
 		(diameter 0)
@@
 	)
 	(junction
-		(at 149.86 228.6)
-		(diameter 0)
-		(color 0 0 0 0)
-	)
-	(junction
 		(at 83.82 280.67)
 		(diameter 0)
@@
 	(wire
 		(pts
+			(xy 149.86 190.5) (xy 149.86 228.6)
+		)
+		(stroke
+			(width 0)
+			(type default)
+		)
+	)
+	(wire
+		(pts
 			(xy 171.45 30.48) (xy 179.07 30.48)
 		)
@@
 	(wire
 		(pts
-			(xy 158.75 228.6) (xy 160.02 228.6)
-		)
-		(stroke
-			(width 0)
-			(type default)
-		)
-	)
-	(wire
-		(pts
 			(xy 388.62 182.88) (xy 388.62 185.42)
 		)
@@
 	(wire
 		(pts
-			(xy 149.86 190.5) (xy 149.86 228.6)
-		)
-		(stroke
-			(width 0)
-			(type default)
-		)
-	)
-	(wire
-		(pts
 			(xy 73.66 68.58) (xy 73.66 81.28)
 		)
@@
 	(wire
 		(pts
-			(xy 151.13 228.6) (xy 149.86 228.6)
-		)
-		(stroke
-			(width 0)
-			(type default)
-		)
-	)
-	(wire
-		(pts
 			(xy 53.34 92.71) (xy 55.88 92.71)
 		)
@@
 	)
 	(symbol
+		(lib_id "linea:WW25WR010FTL")
+		(at 154.94 228.6 0)
+		(unit 1)
+		(exclude_from_sim no)
+		(in_bom yes)
+		(on_board yes)
+		(dnp no)
+		(fields_autoplaced yes)
+		(property "Reference" "R42"
+			(at 154.94 222.25 0)
+			(effects
+				(font
+					(size 1.27 1.27)
+				)
+			)
+		)
+		(property "Value" "WW25WR010FTL"
+			(at 154.94 224.79 0)
+			(effects
+				(font
+					(size 1.27 1.27)
+				)
+			)
+		)
+		(property "Footprint" "linea:R2512"
+			(at 154.94 236.22 0)
+			(effects
+				(font
+					(size 1.27 1.27)
+				)
+				(hide yes)
+			)
+		)
+		(property "Datasheet" "https://lcsc.com/product-detail/Ultra-Low-Resistors-SMD_0-01R-R010-1_C171418.html"
+			(at 154.94 238.76 0)
+			(effects
+				(font
+					(size 1.27 1.27)
+				)
+				(hide yes)
+			)
+		)
+		(property "Description" ""
+			(at 154.94 228.6 0)
+			(effects
+				(font
+					(size 1.27 1.27)
+				)
+				(hide yes)
+			)
+		)
+		(property "LCSC Part" "C171418"
+			(at 154.94 241.3 0)
+			(effects
+				(font
+					(size 1.27 1.27)
+				)
+				(hide yes)
+			)
+		)
+		(pin "1"
+		)
+		(pin "2"
+		)
+		(instances
+			(project ""
+				(path "/f5ca596a-3f37-4a80-af8e-71fb2890766f"
+					(reference "R42")
+					(unit 1)
+				)
+			)
+		)
+	)
+	(symbol
 		(lib_id "linea:EXC14CE900U")
 		(at 97.79 82.55 90)
@@
 					(unit 1)
 				)
-			)
-		)
-	)
-	(symbol
-		(lib_id "Device:R")
-		(at 154.94 228.6 270)
-		(unit 1)
-		(exclude_from_sim no)
-		(in_bom yes)
-		(on_board yes)
-		(dnp no)
-		(property "Reference" "R42"
-			(at 156.718 226.568 90)
-			(effects
-				(font
-					(size 1.27 1.27)
-				)
-				(justify right)
-			)
-		)
-		(property "Value" "10m"
-			(at 156.972 230.886 90)
-			(effects
-				(font
-					(size 1.27 1.27)
-				)
-				(justify right)
-			)
-		)
-		(property "Footprint" "Resistor_SMD:R_0402_1005Metric"
-			(at 154.94 226.822 90)
-			(effects
-				(font
-					(size 1.27 1.27)
-				)
-				(hide yes)
-			)
-		)
-		(property "Datasheet" "~"
-			(at 154.94 228.6 0)
-			(effects
-				(font
-					(size 1.27 1.27)
-				)
-				(hide yes)
-			)
-		)
-		(property "Description" "Resistor"
-			(at 154.94 228.6 0)
-			(effects
-				(font
-					(size 1.27 1.27)
-				)
-				(hide yes)
-			)
-		)
-		(pin "2"
-		)
-		(pin "1"
-		)
-		(instances
-			(project "board"
-				(path "/f5ca596a-3f37-4a80-af8e-71fb2890766f"
-					(reference "R42")
-					(unit 1)
-				)
