File: hardware/board/board.kicad_pcb (KiCad board)
At the start: 4 copper layers, 88 parts, among them J2 Conn_01x26_MountingPin, J3 Conn_01x26_MountingPin, J4 Conn_01x26_MountingPin, Q1 AO3400A, Q2 AO3400A, Q3 AO3400A, U1 STM32WB55RGV6TR, U10 74HC4051, U11 74HC4051, U12 74HC4051, U15 SN74LV1T125DCK, U6 COS8054TR, U7 74HC4051, U8 74HC4051, U9 74HC4051

Commit message: update footprints
Parts:
- removed U15: SN74LV1T125DCK, Package_TO_SOT_SMD:SOT-353_SC-70-5
- added C1: 100nF, Capacitor_SMD:C_0402_1005Metric, F.Cu at (156.8, 69.8)
- added C10: 100nF, Capacitor_SMD:C_0402_1005Metric, F.Cu at (159.7, 71.8)
- added C11: 100nF, Capacitor_SMD:C_0402_1005Metric, F.Cu at (159.7, 73.7)
- added C12: 1uF, Capacitor_SMD:C_0402_1005Metric, F.Cu at (159.7, 75.7)
- added C13: 4.7uF, Capacitor_SMD:C_0402_1005Metric, F.Cu at (159.7, 77.7)
- added C14: 100nF, Capacitor_SMD:C_0402_1005Metric, F.Cu at (159.7, 79.6)
- added C15: 4.7uF, Capacitor_SMD:C_0402_1005Metric, F.Cu at (159.7, 81.6)
- added C16: 0.8pF, Capacitor_SMD:C_0402_1005Metric, F.Cu at (159.7, 83.6)
- added C17: 0.3pF, Capacitor_SMD:C_0402_1005Metric, F.Cu at (162.6, 69.8)
- added C18: 1.5pF, Capacitor_SMD:C_0402_1005Metric, F.Cu at (162.6, 71.8)
- added C19: DNP, Capacitor_SMD:C_0402_1005Metric, F.Cu at (162.6, 73.7)
- added C2: 100nF, Capacitor_SMD:C_0402_1005Metric, F.Cu at (156.8, 71.8)
- added C20: 0.8pF, Capacitor_SMD:C_0402_1005Metric, F.Cu at (162.6, 75.7)
- added C21: 0.3pF, Capacitor_SMD:C_0402_1005Metric, F.Cu at (162.6, 77.7)
- added C3: 100nF, Capacitor_SMD:C_0402_1005Metric, F.Cu at (156.8, 73.7)
- added C4: 100nF, Capacitor_SMD:C_0402_1005Metric, F.Cu at (156.8, 75.7)
- added C5: 4.7pF, Capacitor_SMD:C_0402_1005Metric, F.Cu at (156.8, 77.7)
- added C55: 10uF, Capacitor_SMD:C_0402_1005Metric, F.Cu at (162.6, 79.6)
- added C56: 1uF, Capacitor_SMD:C_0402_1005Metric, F.Cu at (162.6, 81.6)
- added C57: 4.7uF, Capacitor_SMD:C_0402_1005Metric, F.Cu at (162.6, 83.6)
- added C58: 47uF, Capacitor_SMD:C_0402_1005Metric, F.Cu at (165.5, 69.8)
- added C59: 10uF, Capacitor_SMD:C_0402_1005Metric, F.Cu at (165.5, 71.8)
- added C6: 100nF, Capacitor_SMD:C_0402_1005Metric, F.Cu at (156.8, 79.6)
- added C60: 10uF, Capacitor_SMD:C_0402_1005Metric, F.Cu at (165.5, 73.7)
- added C61: 10uF, Capacitor_SMD:C_0402_1005Metric, F.Cu at (165.5, 75.7)
- added C62: 10uF, Capacitor_SMD:C_0402_1005Metric, F.Cu at (165.5, 77.7)
- added C63: 2.2uF, Capacitor_SMD:C_0402_1005Metric, F.Cu at (165.5, 79.6)
- added C64: 470nF, Capacitor_SMD:C_0402_1005Metric, F.Cu at (165.5, 81.6)
- added C65: 1uF, Capacitor_SMD:C_0402_1005Metric, F.Cu at (165.5, 83.6)
- added C66: 1uF, Capacitor_SMD:C_0402_1005Metric, F.Cu at (168.3, 69.8)
- added C67: 2.2uF, Capacitor_SMD:C_0402_1005Metric, F.Cu at (168.3, 71.8)
- added C68: 2.2uF, Capacitor_SMD:C_0402_1005Metric, F.Cu at (168.3, 73.7)
- added C69: 4.7uF, Capacitor_SMD:C_0402_1005Metric, F.Cu at (168.3, 75.7)
- added C7: 1uF, Capacitor_SMD:C_0402_1005Metric, F.Cu at (156.8, 81.6)
- added C70: 10uF, Capacitor_SMD:C_0402_1005Metric, F.Cu at (168.3, 77.7)
- added C71: 10uF, Capacitor_SMD:C_0402_1005Metric, F.Cu at (168.3, 79.6)
- added C8: 10nF, Capacitor_SMD:C_0402_1005Metric, F.Cu at (156.8, 83.6)
- added C9: 1uF, Capacitor_SMD:C_0402_1005Metric, F.Cu at (159.7, 69.8)
- added D1: PESD15VL1BA, PCM_Diode_SMD_AKL:D_SOD-323_TVS, F.Cu at (148.4, 110.6)
- added D2: PESD15VL1BA, PCM_Diode_SMD_AKL:D_SOD-323_TVS, F.Cu at (148.4, 113.8)
- added D3: PESD15VL1BA, PCM_Diode_SMD_AKL:D_SOD-323_TVS, F.Cu at (148.4, 116.9)
- added D4: PESD15VL1BA, PCM_Diode_SMD_AKL:D_SOD-323_TVS, F.Cu at (148.4, 120.0)
- added FL1: ~, linea:FILTET-SMD_0603-6P-L1.6-W0.8-P0.50_LFL182G45TC1A108, F.Cu at (183.5, 89.6)
- added J1: USB_C_Receptacle, USB-C-Power-tester:TYPE-C-31-M-17, F.Cu at (175.1, 96.2)
- added J5: Conn_01x03, Connector_JST:JST_EH_S3B-EH_1x03_P2.50mm_Horizontal, F.Cu at (173.3, 88.5)
- added J6: Conn_01x03_Pin, PCM_4ms_Connector:Pins_1x03_2.54mm_TH, F.Cu at (161.4, 89.1)
- added J7: Conn_01x03_Pin, PCM_4ms_Connector:Pins_1x03_2.54mm_TH, F.Cu at (165.5, 89.1)
- added L1: 10uH, Inductor_SMD:L_0603_1608Metric, F.Cu at (157.4, 85.8)
- added L2: 2.7nH, Inductor_SMD:L_0603_1608Metric, F.Cu at (157.4, 88.3)
- added L3: 3nH, Inductor_SMD:L_0603_1608Metric, F.Cu at (157.4, 90.8)
- added L4: 1uH, Inductor_SMD:L_0603_1608Metric, F.Cu at (157.4, 93.3)
- added L5: 470nH, Inductor_SMD:L_0603_1608Metric, F.Cu at (157.4, 95.8)
- added L6: 470nH, Inductor_SMD:L_0603_1608Metric, F.Cu at (157.4, 98.4)
- added Q4: ~, linea:SOT-523-3_L1.6-W0.8-P1.00-LS1.6-BR, F.Cu at (185.7, 70.3)
- added Q5: ~, linea:SOT-363_L2.0-W1.3-P0.65-LS2.1-BL, F.Cu at (183.9, 82.6)
- added Q6: ~, linea:SOT-23-3_L2.9-W1.3-P1.90-LS2.4-BR, F.Cu at (182.5, 93.2)
- added R1: 5.1K, Resistor_SMD:R_0402_1005Metric, F.Cu at (171.2, 69.8)
- added R10: 10K, Resistor_SMD:R_0402_1005Metric, F.Cu at (174.1, 75.8)
- added R11: 10K, Resistor_SMD:R_0402_1005Metric, F.Cu at (174.1, 77.8)
- added R2: 5.1K, Resistor_SMD:R_0402_1005Metric, F.Cu at (171.2, 71.8)
- added R3: 22, Resistor_SMD:R_0402_1005Metric, F.Cu at (171.2, 73.8)
- added R31: 1.5K, Resistor_SMD:R_0402_1005Metric, F.Cu at (174.1, 79.7)
- added R32: 1.5K, Resistor_SMD:R_0402_1005Metric, F.Cu at (177.0, 69.8)
- added R33: 4.7K, Resistor_SMD:R_0402_1005Metric, F.Cu at (177.0, 71.8)
- added R34: 10K, Resistor_SMD:R_0402_1005Metric, F.Cu at (177.0, 73.8)
- added R35: 100, Resistor_SMD:R_0402_1005Metric, F.Cu at (177.0, 75.8)
- added R36: 10K, Resistor_SMD:R_0402_1005Metric, F.Cu at (177.0, 77.8)
- added R37: 470, Resistor_SMD:R_0402_1005Metric, F.Cu at (177.0, 79.7)
- added R38: 30.1K, Resistor_SMD:R_0402_1005Metric, F.Cu at (179.9, 69.8)
- added R39: 5.23K, Resistor_SMD:R_0402_1005Metric, F.Cu at (179.9, 71.8)
- added R4: 22, Resistor_SMD:R_0402_1005Metric, F.Cu at (171.2, 75.8)
- added R40: 10K, Resistor_SMD:R_0402_1005Metric, F.Cu at (179.9, 73.8)
- added R41: 10K, Resistor_SMD:R_0402_1005Metric, F.Cu at (179.9, 75.8)
- added R42: 10m, Resistor_SMD:R_0402_1005Metric, F.Cu at (179.9, 77.8)
- added R43: DNP, Resistor_SMD:R_0402_1005Metric, F.Cu at (179.9, 79.7)
- added R44: 1.5, Resistor_SMD:R_0402_1005Metric, F.Cu at (182.9, 69.8)
- added R45: 1.5, Resistor_SMD:R_0402_1005Metric, F.Cu at (182.9, 71.8)
- added R46: 3.3, Resistor_SMD:R_0402_1005Metric, F.Cu at (182.9, 73.8)
- added R47: 3.3, Resistor_SMD:R_0402_1005Metric, F.Cu at (182.9, 75.8)
- added R48: 100K, Resistor_SMD:R_0402_1005Metric, F.Cu at (182.9, 77.8)
- added R49: 100K, Resistor_SMD:R_0402_1005Metric, F.Cu at (182.9, 79.7)
- added R5: 0, Resistor_SMD:R_0402_1005Metric, F.Cu at (171.2, 77.8)
- added R6: DNP, Resistor_SMD:R_0402_1005Metric, F.Cu at (171.2, 79.7)
- added R7: DNP, Resistor_SMD:R_0402_1005Metric, F.Cu at (174.1, 69.8)
- added R8: DNP, Resistor_SMD:R_0402_1005Metric, F.Cu at (174.1, 71.8)
- added R9: 10K, Resistor_SMD:R_0402_1005Metric, F.Cu at (174.1, 73.8)
- added U13: SN74LV1T125DCKR, linea:SC-70-5_L2.1-W1.3-P0.65-LS2.1-TL, F.Cu at (182.4, 97.3)
- added U2: ~, linea:QFN-24_L4.0-W4.0-P0.50-TL-EP2.7, F.Cu at (162.4, 96.4)
- added U3: ~, linea:SOT-23-3_L2.9-W1.6-P1.90-LS2.8-BR, F.Cu at (167.4, 95.8)
- added U4: ~, linea:DSBGA-9_L1.7-W1.6-R3-C3-P0.50-BL, F.Cu at (183.3, 86.0)
- added U5: ~, linea:DSBGA-6_L1.4-W1.1-R3-C2-P0.40-BL, F.Cu at (166.7, 99.2)
- C22, C23, C24, C25: footprint Capacitor_SMD:C_0402_1005Metric_Pad0.74x0.62mm_HandSolder -> Capacitor_SMD:C_0402_1005Metric
- C31, C37, C38, C40, C41: footprint Capacitor_SMD:C_0603_1608Metric -> Capacitor_SMD:C_0402_1005Metric
Connections:
- U1 pad 38: /~{E4} -> unconnected-(U1-PB0-Pad38)
- U1 pad 39: /~{E3} -> unconnected-(U1-PB1-Pad39)
- U1 pad 56: unconnected-(U1-PA14-Pad56) -> /S2
- U1 pad 57: unconnected-(U1-PA15-Pad57) -> /S1
- U1 pad 58: unconnected-(U1-PC10-Pad58) -> /S0
- U1 pad 61: unconnected-(U1-PD0-Pad61) -> /~{E4}
- U1 pad 62: unconnected-(U1-PD1-Pad62) -> /~{E3}

Commit message: fnished shcamtic
Parts:
- added SW1: SW_Push, Button_Switch_SMD:SW_SPST_CK_RS282G05A3, F.Cu at (165.7, 56.8)
- added SW2: SW_Push, Button_Switch_SMD:SW_SPST_CK_RS282G05A3, F.Cu at (165.7, 61.9)
- added SW3: SKRTLAE010, linea:KEY-SMD_SKRTLAE010, F.Cu at (174.2, 69.1)
- added X1: XL7EL89CKI-111YLC-32M, linea:CRYSTAL-SMD_4P-L2.0-W1.6-BL, F.Cu at (182.5, 66.5)
- added X2: FC-12M32.768KHZ7PF20PPM, linea:FC-12M_L2.0-W1.2, F.Cu at (173.3, 73.1)
- C37, C38, C40, C41: footprint Capacitor_SMD:C_0402_1005Metric -> Capacitor_SMD:C_0603_1608Metric
- J1: footprint USB-C-Power-tester:TYPE-C-31-M-17 -> Connector_USB:USB_C_Receptacle_Amphenol_12401548E4-2A
- moved J2 156.6 mm to (274.2, 35.8), turned to 180 degrees
- moved J4 131.1 mm to (246.8, 50.4), turned to -90 degrees
- moved J3 124.8 mm to (246.8, 81.8), turned to -90 degrees
- moved D2 77.5 mm to (186.4, 46.2)
- moved D1 77.5 mm to (186.4, 43.1)
- moved D3 77.5 mm to (186.4, 49.3)
- moved D4 77.5 mm to (186.4, 52.5)
- moved U7 55.6 mm to (162.7, 38.7)
- moved U8 55.6 mm to (167.4, 38.7)
- moved U9 55.6 mm to (172.2, 38.7)
- moved U10 55.6 mm to (176.9, 38.7)
- moved U11 55.6 mm to (181.7, 38.7)
- moved U12 55.6 mm to (186.4, 38.7)
- moved J1 49.1 mm to (166.2, 47.9)
- moved C49 47.3 mm to (153.1, 36.8)
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Connections:
- J2 pad 1: unconnected-(J2-Pin_1-Pad1) -> /Y0
- J2 pad 10: /Y13 -> /Y7
- J2 pad 11: /Y12 -> /Y8
- J2 pad 12: /Y11 -> /Y9
- J2 pad 13: /Y10 -> GND
- J2 pad 14: GND -> /Y10
- J2 pad 15: /Y9 -> /Y11
- J2 pad 16: /Y8 -> /Y12
- J2 pad 17: /Y7 -> /Y13
- J2 pad 18: /Y6 -> GND
- J2 pad 19: GND -> /Y14
- J2 pad 2: unconnected-(J2-Pin_2-Pad2) -> /Y1
- J2 pad 20: /Y5 -> /Y15
- J2 pad 21: /Y4 -> /Y16
- J2 pad 22: /Y3 -> /Y17
- J2 pad 23: /Y2 -> GND
- J2 pad 24: GND -> unconnected-(J2-Pin_24-Pad24)
- J2 pad 25: /Y1 -> unconnected-(J2-Pin_25-Pad25)
- J2 pad 26: /Y0 -> unconnected-(J2-Pin_26-Pad26)
- J2 pad 3: unconnected-(J2-Pin_3-Pad3) -> GND
- J2 pad 4: GND -> /Y2
- J2 pad 5: /Y17 -> /Y3
- J2 pad 6: /Y16 -> /Y4
- J2 pad 7: /Y15 -> /Y5
- J2 pad 8: /Y14 -> GND
- J2 pad 9: GND -> /Y6
- J3 pad 1: unconnected-(J3-Pin_1-Pad1) -> /X20
- J3 pad 10: unconnected-(J3-Pin_10-Pad10) -> /X27
- J3 pad 13: unconnected-(J3-Pin_13-Pad13) -> GND
- J3 pad 14: GND -> unconnected-(J3-Pin_14-Pad14)
- J3 pad 17: /X27 -> unconnected-(J3-Pin_17-Pad17)
- J3 pad 18: /X26 -> GND
- J3 pad 19: GND -> unconnected-(J3-Pin_19-Pad19)
- J3 pad 2: unconnected-(J3-Pin_2-Pad2) -> /X21
- J3 pad 20: /X25 -> unconnected-(J3-Pin_20-Pad20)
- J3 pad 21: /X24 -> unconnected-(J3-Pin_21-Pad21)
- J3 pad 22: /X23 -> unconnected-(J3-Pin_22-Pad22)
- J3 pad 23: /X22 -> GND
- J3 pad 24: GND -> unconnected-(J3-Pin_24-Pad24)
- J3 pad 25: /X21 -> unconnected-(J3-Pin_25-Pad25)
- J3 pad 26: /X20 -> unconnected-(J3-Pin_26-Pad26)
- J3 pad 3: unconnected-(J3-Pin_3-Pad3) -> GND
- J3 pad 4: GND -> /X22
- J3 pad 5: unconnected-(J3-Pin_5-Pad5) -> /X23
- J3 pad 6: unconnected-(J3-Pin_6-Pad6) -> /X24
- J3 pad 7: unconnected-(J3-Pin_7-Pad7) -> /X25
- J3 pad 8: unconnected-(J3-Pin_8-Pad8) -> GND
- J3 pad 9: GND -> /X26
- J4 pad 1: unconnected-(J4-Pin_1-Pad1) -> /X0
- J4 pad 10: /X13 -> /X7
- J4 pad 11: /X12 -> /X8
- J4 pad 12: /X11 -> /X9
- J4 pad 13: /X10 -> GND
- J4 pad 14: GND -> /X10
- J4 pad 15: /X9 -> /X11
- J4 pad 16: /X8 -> /X12
- J4 pad 17: /X7 -> /X13
- J4 pad 18: /X6 -> GND
- J4 pad 19: GND -> /X14
- J4 pad 2: /X19 -> /X1
- J4 pad 20: /X5 -> /X15
- J4 pad 21: /X4 -> /X16
- J4 pad 22: /X3 -> /X17
- J4 pad 23: /X2 -> GND
- J4 pad 24: GND -> /X18
- J4 pad 25: /X1 -> /X19
- J4 pad 26: /X0 -> unconnected-(J4-Pin_26-Pad26)
- J4 pad 3: /X18 -> GND
- J4 pad 4: GND -> /X2
- J4 pad 5: /X17 -> /X3
- J4 pad 6: /X16 -> /X4
- J4 pad 7: /X15 -> /X5
- J4 pad 8: /X14 -> GND
- J4 pad 9: GND -> /X6
Routing:
- net GND: track 0.00 -> 67.1 mm, vias 0 -> 29
- net /X22: track 0.00 -> 7.91 mm
- net unconnected-(J3-Pin_12-Pad12): track 0.00 -> 4.11 mm
- net unconnected-(J3-Pin_16-Pad16): track 0.00 -> 3.94 mm
- net /X21: track 0.00 -> 3.87 mm
- net /X27: track 0.00 -> 2.35 mm
- net /X1: track 0.00 -> 2.22 mm
- net /X0: track 0.00 -> 2.18 mm
- net unconnected-(J3-Pin_11-Pad11): track 0.00 -> 2.16 mm
- net /Y10: track 0.00 -> 2.15 mm
- net /Y11: track 0.00 -> 2.12 mm
- net /Y12: track 0.00 -> 2.05 mm
- net /X4: track 0.00 -> 1.89 mm
- net /X26: track 0.00 -> 1.84 mm
- net /X6: track 0.00 -> 1.73 mm
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- added copper zone on B.Cu, net GND
- added copper zone on F.Cu, net GND
- added copper zone on In1.Cu, net GND
- added copper zone on In2.Cu, net GND
Other:
- board outline added: 45 x 60 mm

Commit message: added touches
Parts:
- U10, U11, U12, U7, U8, U9: footprint Package_DFN_QFN:DHVQFN-16-1EP_2.5x3.5mm_P0.5mm_EP1x2mm -> Package_SO:TSSOP-16_4.4x5mm_P0.65mm
- moved J2 212.3 mm to (70.9, 96.9)
- moved J4 174.9 mm to (98.3, 142.9), turned to 90 degrees
- moved J3 152.3 mm to (97.2, 110.6), turned to 90 degrees
- moved U11 130.7 mm to (68.7, 104.4)
- moved J1 101.2 mm to (265.6, 28.8), turned to 180 degrees
- moved U1 87.7 mm to (250.1, 92.2)
- moved J5 81.0 mm to (248.5, 84.5)
- moved SW3 73.3 mm to (247.3, 63.9)
- moved R25 62.1 mm to (127.8, 32.7)
- moved C34 61.7 mm to (188.8, 48.7)
- moved U2 58.5 mm to (135.8, 36.7)
- moved D8 57.8 mm to (168.8, 34.7)
- moved D1 57.7 mm to (135.8, 70.7)
- moved D11 57.6 mm to (168.8, 43.7)
- moved U4 57.3 mm to (131.8, 37.7)
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Connections:
- U10 pad 1: /Y0 -> /X26
- U10 pad 12: /X27 -> /X22
- U10 pad 13: /X24 -> /X23
- U10 pad 14: /X25 -> /X24
- U10 pad 15: /X26 -> /X25
- U10 pad 2: /Y2 -> /X27
- U10 pad 4: /Y3 -> unconnected-(U10-A7-Pad4)
- U10 pad 5: /Y1 -> unconnected-(U10-A5-Pad5)
- U11 pad 1: /Y8 -> /Y7
- U11 pad 12: /Y7 -> /Y3
- U11 pad 13: /Y4 -> /Y2
- U11 pad 14: /Y5 -> /Y1
- U11 pad 15: /Y6 -> /Y0
- U11 pad 2: /Y10 -> /Y6
- U11 pad 4: /Y11 -> /Y5
- U11 pad 5: /Y9 -> /Y4
- U12 pad 1: /Y16 -> /Y12
- U12 pad 12: /Y15 -> /Y8
- U12 pad 13: /Y12 -> /Y9
- U12 pad 14: /Y13 -> /Y10
- U12 pad 15: /Y14 -> /Y11
- U12 pad 2: unconnected-(U12-A6-Pad2) -> /Y13
- U12 pad 4: unconnected-(U12-A7-Pad4) -> /Y14
- U12 pad 5: /Y17 -> /Y15
- U7 pad 1: /X4 -> /X2
- U7 pad 12: /X3 -> /Y16
- U7 pad 13: /X0 -> /Y17
- U7 pad 14: /X1 -> /X0
- U7 pad 15: /X2 -> /X1
- U7 pad 2: /X6 -> /X3
- U7 pad 4: /X7 -> /X4
- U8 pad 1: /X12 -> /X10
- U8 pad 12: /X11 -> /X6
- U8 pad 13: /X8 -> /X7
- U8 pad 14: /X9 -> /X8
- U8 pad 15: /X10 -> /X9
- U8 pad 2: /X14 -> /X11
- U8 pad 4: /X15 -> /X12
- U9 pad 1: /X20 -> /X18
- U9 pad 12: /X19 -> /X14
- U9 pad 13: /X16 -> /X15
- U9 pad 14: /X17 -> /X16
- U9 pad 15: /X18 -> /X17
- U9 pad 2: /X22 -> /X19
- U9 pad 4: /X23 -> /X20
Routing:
- net GND: track 67.1 -> 0.00 mm, vias 29 -> 0
- net /X22: track 7.91 -> 0.00 mm
- net unconnected-(J3-Pin_12-Pad12): track 4.11 -> 0.00 mm
- net unconnected-(J3-Pin_16-Pad16): track 3.94 -> 0.00 mm
- net /X21: track 3.87 -> 0.00 mm
- net /X27: track 2.35 -> 0.00 mm
- net /X1: track 2.22 -> 0.00 mm
- net /X0: track 2.18 -> 0.00 mm
- net unconnected-(J3-Pin_11-Pad11): track 2.16 -> 0.00 mm
- net /Y10: track 2.15 -> 0.00 mm
- net /Y11: track 2.12 -> 0.00 mm
- net /Y12: track 2.05 -> 0.00 mm
- net /X4: track 1.89 -> 0.00 mm
- net /X26: track 1.84 -> 0.00 mm
- net /X6: track 1.73 -> 0.00 mm
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- removed copper zone on B.Cu, net GND
- removed copper zone on F.Cu, net GND
- removed copper zone on In1.Cu, net GND
- removed copper zone on In2.Cu, net GND
Other:
- board size 45 x 60 mm -> 73.2 x 60 mm

Commit message: pcb power start
Parts:
- removed D1, D2: PESD15VL1BA, PCM_Diode_SMD_AKL:D_SOD-323_TVS
- removed J1: USB_C_Receptacle, Connector_USB:USB_C_Receptacle_Amphenol_12401548E4-2A
- removed R3, R4: 22, Resistor_SMD:R_0402_1005Metric
- added L8: EXC14CE900U, linea:FILTER-SMD_4P-L0.9-W0.7-P0.50-BL, F.Cu at (41.5, 103.5)
- added U14: USBLC6-2P6, Package_TO_SOT_SMD:SOT-666, F.Cu at (41.5, 101.2)
- added USB1: TYPE-C 16PIN 2MD(073), linea:USB-C-SMD_TYPE-C-6PIN-2MD-073, F.Cu at (41.6, 96.1)
- moved J5 350.7 mm to (-97.6, 141.2), turned to 90 degrees
- moved U1 212.3 mm to (38.5, 109.5)
- moved C67 175.4 mm to (-14.8, 127.0), turned to 90 degrees
- moved U5 174.6 mm to (-16.4, 127.0)
- moved C68 172.4 mm to (-19.4, 135.8)
- moved C69 172.4 mm to (-19.4, 136.8)
- moved C70 172.4 mm to (-24.4, 128.8)
- moved C71 172.4 mm to (0.55, 122.8)
- moved L5 172.4 mm to (-18.4, 133.8)
- moved L6 172.4 mm to (-18.4, 130.8)
- moved R44 172.4 mm to (-16.4, 137.8)
- moved R45 172.4 mm to (-16.4, 135.8)
- moved R46 172.4 mm to (-13.4, 130.8)
- moved R47 172.4 mm to (-13.4, 131.8)
- moved C55 134.2 mm to (33.6, 27.2)
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Connections:
- J2 pad 1: /Y0 -> unconnected-(J2-Pin_1-Pad1)
- J2 pad 10: /Y7 -> /Y13
- J2 pad 11: /Y8 -> /Y12
- J2 pad 12: /Y9 -> /Y11
- J2 pad 13: GND -> /Y10
- J2 pad 14: /Y10 -> GND
- J2 pad 15: /Y11 -> /Y9
- J2 pad 16: /Y12 -> /Y8
- J2 pad 17: /Y13 -> /Y7
- J2 pad 18: GND -> /Y6
- J2 pad 19: /Y14 -> GND
- J2 pad 2: /Y1 -> unconnected-(J2-Pin_2-Pad2)
- J2 pad 20: /Y15 -> /Y5
- J2 pad 21: /Y16 -> /Y4
- J2 pad 22: /Y17 -> /Y3
- J2 pad 23: GND -> /Y2
- J2 pad 24: unconnected-(J2-Pin_24-Pad24) -> GND
- J2 pad 25: unconnected-(J2-Pin_25-Pad25) -> /Y1
- J2 pad 26: unconnected-(J2-Pin_26-Pad26) -> /Y0
- J2 pad 3: GND -> unconnected-(J2-Pin_3-Pad3)
- J2 pad 4: /Y2 -> GND
- J2 pad 5: /Y3 -> /Y17
- J2 pad 6: /Y4 -> /Y16
- J2 pad 7: /Y5 -> /Y15
- J2 pad 8: GND -> /Y14
- J2 pad 9: /Y6 -> GND
- J3 pad 1: /X20 -> unconnected-(J3-Pin_1-Pad1)
- J3 pad 10: /X27 -> /X13
- J3 pad 11: unconnected-(J3-Pin_11-Pad11) -> /X12
- J3 pad 12: unconnected-(J3-Pin_12-Pad12) -> /X11
- J3 pad 13: GND -> /X10
- J3 pad 14: unconnected-(J3-Pin_14-Pad14) -> GND
- J3 pad 15: unconnected-(J3-Pin_15-Pad15) -> /X9
- J3 pad 16: unconnected-(J3-Pin_16-Pad16) -> /X8
- J3 pad 17: unconnected-(J3-Pin_17-Pad17) -> /X7
- J3 pad 18: GND -> /X6
- J3 pad 19: unconnected-(J3-Pin_19-Pad19) -> GND
- J3 pad 2: /X21 -> /X19
- J3 pad 20: unconnected-(J3-Pin_20-Pad20) -> /X5
- J3 pad 21: unconnected-(J3-Pin_21-Pad21) -> /X4
- J3 pad 22: unconnected-(J3-Pin_22-Pad22) -> /X3
- J3 pad 23: GND -> /X2
- J3 pad 24: unconnected-(J3-Pin_24-Pad24) -> GND
- J3 pad 25: unconnected-(J3-Pin_25-Pad25) -> /X1
- J3 pad 26: unconnected-(J3-Pin_26-Pad26) -> /X0
- J3 pad 3: GND -> /X18
- J3 pad 4: /X22 -> GND
- J3 pad 5: /X23 -> /X17
- J3 pad 6: /X24 -> /X16
- J3 pad 7: /X25 -> /X15
- J3 pad 8: GND -> /X14
- J3 pad 9: /X26 -> GND
- J4 pad 1: /X0 -> unconnected-(J4-Pin_1-Pad1)
- J4 pad 10: /X7 -> unconnected-(J4-Pin_10-Pad10)
- J4 pad 11: /X8 -> unconnected-(J4-Pin_11-Pad11)
- J4 pad 12: /X9 -> unconnected-(J4-Pin_12-Pad12)
- J4 pad 13: GND -> unconnected-(J4-Pin_13-Pad13)
- J4 pad 14: /X10 -> GND
- J4 pad 15: /X11 -> unconnected-(J4-Pin_15-Pad15)
- J4 pad 16: /X12 -> unconnected-(J4-Pin_16-Pad16)
- J4 pad 17: /X13 -> /X27
- J4 pad 18: GND -> /X26
- J4 pad 19: /X14 -> GND
- J4 pad 2: /X1 -> unconnected-(J4-Pin_2-Pad2)
- J4 pad 20: /X15 -> /X25
- J4 pad 21: /X16 -> /X24
- J4 pad 22: /X17 -> /X23
- J4 pad 23: GND -> /X22
- J4 pad 24: /X18 -> GND
- J4 pad 25: /X19 -> /X21
- J4 pad 26: unconnected-(J4-Pin_26-Pad26) -> /X20
- J4 pad 3: GND -> unconnected-(J4-Pin_3-Pad3)
- J4 pad 4: /X2 -> GND
- J4 pad 5: /X3 -> unconnected-(J4-Pin_5-Pad5)
- J4 pad 6: /X4 -> unconnected-(J4-Pin_6-Pad6)
- J4 pad 7: /X5 -> unconnected-(J4-Pin_7-Pad7)
- J4 pad 8: GND -> unconnected-(J4-Pin_8-Pad8)
- J4 pad 9: /X6 -> GND
- U11 pad 1: /Y7 -> /Y4
- U11 pad 12: /Y3 -> /Y0
- U11 pad 13: /Y2 -> /Y1
- U11 pad 14: /Y1 -> /Y2
- U11 pad 15: /Y0 -> /Y3
- U11 pad 2: /Y6 -> /Y5
- U11 pad 4: /Y5 -> /Y6
- U11 pad 5: /Y4 -> /Y7
Routing:
- net VBUS: track 0.00 -> 13.0 mm
- net GND: vias 0 -> 1

Commit message: bunch o f stuff
Parts:
- removed C16: 0.8pF, Capacitor_SMD:C_0402_1005Metric
- removed C17: 0.3pF, Capacitor_SMD:C_0402_1005Metric
- removed C18: 1.5pF, Capacitor_SMD:C_0402_1005Metric
- removed C19: DNP, Capacitor_SMD:C_0402_1005Metric
- removed C46, C47: 100nF, Capacitor_SMD:C_0402_1005Metric
- removed FL1: ~, linea:FILTET-SMD_0603-6P-L1.6-W0.8-P0.50_LFL182G45TC1A108
- removed J6, J7: Conn_01x03_Pin, PCM_4ms_Connector:Pins_1x03_2.54mm_TH
- removed L2: 2.7nH, Inductor_SMD:L_0603_1608Metric
- removed L3: 3nH, Inductor_SMD:L_0603_1608Metric
- removed R5: 0, Resistor_SMD:R_0402_1005Metric
- removed R6, R7, R8: DNP, Resistor_SMD:R_0402_1005Metric
- added AE1: 2450AT18A100E, linea:ANT-SMD_L3.2-W1.6, F.Cu at (59.4, 147.3)
- added D1: 1N4148WT, Diode_SMD:D_SOD-523, F.Cu at (90.1, 150.0)
- added FL2: MLPF-WB55-01E3, linea:FILTER-SMD_6P-L1.6-W1.0-P0.50-BL, F.Cu at (73.2, 133.0)
- added L9: 470nH, Inductor_SMD:L_Murata_DFE201610P, F.Cu at (87.7, 163.7)
- added TP1: TestPoint, TestPoint:TestPoint_Pad_1.5x1.5mm, F.Cu at (65.7, 170.8)
- added TP2: TestPoint, TestPoint:TestPoint_Pad_1.5x1.5mm, F.Cu at (63.0, 170.8)
- added TP3: TestPoint, TestPoint:TestPoint_Pad_1.5x1.5mm, F.Cu at (60.4, 170.8)
- added U15: FAN48610BUC50X, linea:WLCSP-9_L1.2-W1.2-R3-C3-P0.40-BL, F.Cu at (88.1, 165.6)
- C44: value 100nF -> 10uF
- C45: value 100nF -> 22uF
- moved SW3 180.1 mm to (100.9, 168.7), turned to 90 degrees
- moved J5 175.2 mm to (76.0, 165.2), turned to 180 degrees
- moved R31 160.9 mm to (86.2, 157.1), turned to -90 degrees
- moved R40 156.6 mm to (76.8, 160.1), turned to -90 degrees
- moved R39 154.7 mm to (79.5, 153.6)
- moved R41 154.6 mm to (78.7, 157.0), turned to 180 degrees
- moved C60 151.4 mm to (78.2, 159.3), turned to 90 degrees
- moved U2 146.4 mm to (82.8, 157.1), turned to 180 degrees
- moved R30 146.3 mm to (65.8, 124.2), turned to 180 degrees
- moved U4 144.7 mm to (76.2, 157.7), turned to 90 degrees
- moved C57 143.5 mm to (83.6, 161.0), turned to -90 degrees
- moved R29 143.4 mm to (65.8, 125.2)
- moved C55 143.0 mm to (85.3, 160.5)
- moved C34 141.5 mm to (65.7, 118.5), turned to 90 degrees
- moved SW1 141.1 mm to (62.8, 165.2), turned to 180 degrees
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Connections:
- net Net-(U1-PA11) renamed /D+
- net Net-(U1-PA12) renamed /D-
- C11 pad 1: Net-(U1-VDDRF) -> +3.3V
- C12 pad 1: Net-(U1-VDDRF) -> +3.3V
- C44 pad 1: VSSA -> SYS
- C44 pad 2: VBUS -> GND
- C45 pad 1: VEE -> +5V
- C45 pad 2: VSSA -> GND
- C48 pad 2: VBUS -> +5V
- C50 pad 2: VBUS -> +5V
- C52 pad 2: VBUS -> +5V
- C56 pad 1: +5V -> USB_5V
- J2 pad 14: GND -> GNDS
- J2 pad 19: GND -> GNDS
- J2 pad 24: GND -> GNDS
- J2 pad 4: GND -> GNDS
- J2 pad 9: GND -> GNDS
- J3 pad 14: GND -> GNDS
- J3 pad 19: GND -> GNDS
- J3 pad 24: GND -> GNDS
- J3 pad 4: GND -> GNDS
- J3 pad 9: GND -> GNDS
- J4 pad 14: GND -> GNDS
- J4 pad 19: GND -> GNDS
- J4 pad 24: GND -> GNDS
- J4 pad 4: GND -> GNDS
- J4 pad 9: GND -> GNDS
- JP1 pad 1: GND -> GNDS
- Q5 pad 2: VBUS -> Net-(D1-A)
- Q5 pad 3: VBUS -> Net-(Q5-C2)
- Q5 pad 4: +5V -> USB_5V
- Q5 pad 5: VBUS -> Net-(D1-A)
- Q6 pad 2: +5V -> USB_5V
- R48 pad 1: VBUS -> Net-(Q5-C2)
- U1 pad 24: /TX -> unconnected-(U1-PA9-Pad24)
- U1 pad 33: Net-(U1-VDDRF) -> +3.3V
- U1 pad 67: /RX -> unconnected-(U1-PB7-Pad67)
- U10 pad 16: VBUS -> +5V
- U11 pad 16: VBUS -> +5V
- U12 pad 16: VBUS -> +5V
- U2 pad 1: +5V -> USB_5V
- U7 pad 16: VBUS -> +5V
- U8 pad 16: VBUS -> +5V
- U9 pad 16: VBUS -> +5V
Routing:
- net VSSA: track 0.00 -> 186.9 mm, vias 0 -> 57
- net +3.3V: track 0.00 -> 156.2 mm, vias 0 -> 13
- net VEE: track 0.00 -> 130.0 mm, vias 0 -> 7
- net GND: track 0.00 -> 129.9 mm, vias 1 -> 151
- net +5V: track 0.00 -> 116.8 mm, vias 0 -> 11
- net /S2: track 0.00 -> 104.3 mm, vias 0 -> 7
- net /S1: track 0.00 -> 101.1 mm, vias 0 -> 7
- net /S0: track 0.00 -> 100.7 mm, vias 0 -> 7
- net GNDS: track 0.00 -> 97.6 mm, vias 0 -> 17
- net /ABUS: track 0.00 -> 88.2 mm, vias 0 -> 7
- net /~{E4}: track 0.00 -> 80.5 mm, vias 0 -> 2
- net /~{E5}: track 0.00 -> 73.6 mm, vias 0 -> 2
- net /~{E0}: track 0.00 -> 61.4 mm, vias 0 -> 2
- net RESET: track 0.00 -> 61.2 mm, vias 0 -> 3
- net /EXCITER: track 0.00 -> 50.9 mm, vias 0 -> 2
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- added copper zone on B.Cu, net (none)
- added copper zone on F.Cu, net (none)
- added copper zone on In1.Cu, net (none)
- added copper zone on In2.Cu, net (none)
- added copper zone on B.Cu, net GND
- added copper zone on F.Cu, net GND
- added copper zone on In1.Cu, net GND
- added copper zone on In2.Cu, net GND
- added copper zone on B.Cu, net VSSA
- added copper zone on F.Cu, net VSSA
- added copper zone on In1.Cu, net VSSA
- added copper zone on In2.Cu, net VSSA
Other:
- board size 73.2 x 60 mm -> 45 x 80 mm
- board text added: "Linea V1"
