File: hardware/board/board.kicad_pcb (KiCad board)
At the start: 4 copper layers, 45 x 80 mm, 174 parts, among them J2 Conn_01x26_MountingPin, J3 Conn_01x26_MountingPin, J4 Conn_01x26_MountingPin, J5 Conn_01x03, Q1 AO3400A, Q2 AO3400A, Q3 AO3400A, SW1 SW_Push, SW2 SW_Push, SW3 SKRTLAE010, U1 STM32WB55RGV6TR, U10 74HC4051, U11 74HC4051, U12 74HC4051, U13 SN74LV1T125DCKR, U14 USBLC6-2P6, U15 FAN48610BUC50X, U6 COS8054TR, U7 74HC4051, U8 74HC4051, U9 74HC4051, X1 XL7EL89CKI-111YLC-32M, X2 FC-12M32.768KHZ7PF20PPM

Commit message: finished board
Parts:
- removed C54: 72nF, Capacitor_SMD:C_0402_1005Metric
- removed U3: ~, linea:SOT-23-3_L2.9-W1.6-P1.90-LS2.8-BR
- added C16: 3.9nF, Capacitor_SMD:C_0402_1005Metric, F.Cu at (85.5, 114.2)
- added C17: 3.6nF, Capacitor_SMD:C_0603_1608Metric, F.Cu at (85.1, 118.5)
- added C18: 68nF, Capacitor_SMD:C_0402_1005Metric, F.Cu at (78.2, 145.2)
- added C19: 3.9nF, Capacitor_SMD:C_0402_1005Metric, F.Cu at (78.2, 144.2)
- added U16: RS3221-3.3YUTDN4, linea:UTDFN-4_L1.0-W1.0-P0.63-BL-EP-1, F.Cu at (76.6, 151.4)
- C27: value 7.2nF -> 3.6nF; footprint Capacitor_SMD:C_0402_1005Metric -> Capacitor_SMD:C_0603_1608Metric
- C58: value 47uF -> 47nF
- C73: value 72nF -> 68nF
- U1: value STM32WB55RGV6TR -> STM32WB55RGV6
- moved C26 2.42 mm to (82.5, 116.5), turned to 180 degrees
- moved C27 1.92 mm to (85.0, 116.9)
- moved L7 1.79 mm to (85.6, 112.3), turned to 0 degrees
- moved C73 0.14 mm to (84.4, 114.2)
Routing:
- net Net-(U16-EN): track 11.3 -> 16.4 mm, vias 2 -> 3
- net VSSA: track 186.9 -> 183.4 mm, vias 57 -> 56
- net Net-(C17-Pad2): track 1.39 -> 3.91 mm
- net Net-(C16-Pad2): track 1.81 -> 4.30 mm
- net GND: track 129.9 -> 132.0 mm, vias 151 -> 150
- net +5V: track 116.8 -> 118.6 mm
- net Net-(U13-Y): track 1.35 -> 2.30 mm
- net /ABUS: track 88.2 -> 88.8 mm

Commit message: impdance matching
Parts:
- moved AE1 0.70 mm to (60.1, 147.3)
Routing:
- net VSSA: vias 56 -> 59
- net GND: vias 150 -> 167

Commit message: impdance matching
Parts:
- moved FL2 0.06 mm to (73.2, 133.1)
