File: hardware/board/board.kicad_pcb (KiCad board)
At the start: 4 copper layers, 45 x 80 mm, 177 parts, among them J2 Conn_01x26_MountingPin, J3 Conn_01x26_MountingPin, J4 Conn_01x26_MountingPin, J5 Conn_01x03, Q1 AO3400A, Q2 AO3400A, Q3 AO3400A, SW1 SW_Push, SW2 SW_Push, SW3 SKRTLAE010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

Commit message: esd prtot
Connections:
- L8 pad 3: Net-(USB1-DP1) -> Net-(L8-Pad3)
- L8 pad 4: Net-(USB1-DN1) -> Net-(L8-Pad4)
- U14 pad 4: Net-(USB1-DN1) -> Net-(L8-Pad4)
- U14 pad 6: Net-(USB1-DP1) -> Net-(L8-Pad3)
Routing:
- net Net-(USB1-DN1): track 7.55 -> 4.51 mm
- net Net-(USB1-DP1): track 7.47 -> 4.47 mm
- net Net-(L8-Pad4): track 0.00 -> 1.34 mm
- net Net-(L8-Pad3): track 0.00 -> 1.30 mm
Changed lines of the file:
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@@
 	(net 202 "Net-(C17-Pad2)")
 	(net 203 "Net-(U16-EN)")
+	(net 204 "Net-(L8-Pad4)")
+	(net 205 "Net-(L8-Pad3)")
 	(footprint "Capacitor_SMD:C_0402_1005Metric"
 		(placed yes)
@@
 			(size 0.3 0.3)
 			(layers "F.Cu" "F.Mask" "F.Paste")
-			(net 190 "Net-(USB1-DP1)")
+			(net 205 "Net-(L8-Pad3)")
 			(pinfunction "3")
 			(pintype "unspecified")
@@
 			(size 0.3 0.3)
 			(layers "F.Cu" "F.Mask" "F.Paste")
-			(net 191 "Net-(USB1-DN1)")
+			(net 204 "Net-(L8-Pad4)")
 			(pinfunction "4")
 			(pintype "unspecified")
@@
 			(layers "F.Cu" "F.Mask" "F.Paste")
 			(roundrect_rratio 0.25)
-			(net 191 "Net-(USB1-DN1)")
+			(net 204 "Net-(L8-Pad4)")
 			(pinfunction "I/O2")
 			(pintype "passive")
@@
 			(layers "F.Cu" "F.Mask" "F.Paste")
 			(roundrect_rratio 0.25)
-			(net 190 "Net-(USB1-DP1)")
+			(net 205 "Net-(L8-Pad3)")
 			(pinfunction "I/O1")
 			(pintype "passive")
@@
 	)
 	(segment
-		(start 93.11 160.2175)
-		(end 92.1475 160.2175)
-		(width 0.25)
-		(layer "F.Cu")
-		(net 190)
-	)
-	(segment
-		(start 94.81 160.2175)
-		(end 93.11 160.2175)
-		(width 0.25)
-		(layer "F.Cu")
-		(net 190)
-	)
-	(segment
 		(start 95.6 160.2)
 		(end 94.8275 160.2)
@@
 	)
 	(segment
-		(start 92.1475 160.2175)
-		(end 91.91 159.98)
-		(width 0.25)
-		(layer "F.Cu")
-		(net 190)
-	)
-	(segment
 		(start 96 159.1)
 		(end 95.675 158.775)
@@
 	)
 	(segment
-		(start 93.11 159.1425)
-		(end 92.2475 159.1425)
-		(width 0.25)
-		(layer "F.Cu")
-		(net 191)
-	)
-	(segment
 		(start 95.4865 159.1425)
 		(end 95.944 159.6)
@@
 	)
 	(segment
-		(start 92.2475 159.1425)
-		(end 91.91 159.48)
-		(width 0.25)
-		(layer "F.Cu")
-		(net 191)
-	)
-	(segment
 		(start 97.45 159.794)
 		(end 97.45 160.5)
@@
 	)
 	(segment
-		(start 94.81 159.1425)
-		(end 93.11 159.1425)
-		(width 0.25)
-		(layer "F.Cu")
-		(net 191)
-	)
-	(segment
 		(start 89.64 151.41)
 		(end 89.64 153.39)
@@
 		(net 203)
 	)
+	(segment
+		(start 93.11 159.1425)
+		(end 92.2475 159.1425)
+		(width 0.25)
+		(layer "F.Cu")
+		(net 204)
+	)
+	(segment
+		(start 92.2475 159.1425)
+		(end 91.91 159.48)
+		(width 0.25)
+		(layer "F.Cu")
+		(net 204)
+	)
+	(segment
+		(start 93.11 160.2175)
+		(end 92.1475 160.2175)
+		(width 0.25)
+		(layer "F.Cu")
+		(net 205)
+	)
+	(segment
+		(start 92.1475 160.2175)
+		(end 91.91 159.98)
+		(width 0.25)
+		(layer "F.Cu")
+		(net 205)
+	)
 	(zone
 		(net 95)
@@
 	)
 	(zone
-		(net 13)
-		(net_name "GND")
-		(layer "F.Cu")
-		(name "$teardrop_padvia$")
-		(hatch none 0.1)
-		(priority 30038)
-		(attr
-			(teardrop
-				(type padvia)
-			)
-		)
-		(connect_pads yes
-			(clearance 0)
-		)
-		(min_thickness 0.0254)
-		(filled_areas_thickness no)
-		(fill yes
-			(thermal_gap 0.5)
-			(thermal_bridge_width 0.5)
-			(island_removal_mode 1)
-			(island_area_min 10)
-		)
-		(polygon
-			(pts
-				(xy 72.6 136.055764) (xy 72.4 136.055764) (xy 72.205764 136.591473) (xy 72.5 136.651) (xy 72.794236 136.591473)
-			)
-		)
-	)
-	(zone
 		(net 97)
 		(net_name "/TIM2_CH2")
@@
 	)
 	(zone
-		(net 27)
-		(net_name "VBUS")
-		(layer "F.Cu")
-		(name "$teardrop_padvia$")
-		(hatch none 0.1)
-		(priority 30178)
-		(attr
-			(teardrop
-				(type padvia)
-			)
-		)
-		(connect_pads yes
-			(clearance 0)
-		)
-		(min_thickness 0.0254)
-		(filled_areas_thickness no)
-		(fill yes
-			(thermal_gap 0.5)
-			(thermal_bridge_width 0.5)
-			(island_removal_mode 1)
-			(island_area_min 10)
-		)
-		(polygon
-			(pts
-				(xy 93.304323 159.58) (xy 93.304323 159.78) (xy 93.706105 159.870677) (xy 93.751 159.65) (xy 93.706105 159.429323)
-			)
-		)
-	)
-	(zone
 		(net 17)
 		(net_name "Net-(C34-Pad1)")
@@
 			)
 		)
-	)
-	(zone
-		(net 13)
-		(net_name "GND")
-		(layer "F.Cu")
-		(name "$teardrop_padvia$")
-		(hatch none 0.1)
-		(priority 30139)
-		(attr
-			(teardrop
-				(type padvia)
-			)
-		)
-		(connect_pads yes
-			(clearance 0)
-		)
-		(min_thickness 0.0254)
-		(filled_areas_thickness no)
-		(fill yes
-			(thermal_gap 0.5)
-			(thermal_bridge_width 0.5)
-			(island_removal_mode 1)
-			(island_area_min 10)
-		)
-		(polygon
-			(pts
-				(xy 94.772625 159.83) (xy 94.772625 159.53) (xy 94.370843 159.454219) (xy 94.325948 159.674896)
-				(xy 94.370843 159.895573)
-			)
-		)
