File: hardware/board/board.kicad_pcb (KiCad board)
At the start: 4 copper layers, 45 x 80 mm, 177 parts, among them J2 Conn_01x26_MountingPin, J3 Conn_01x26_MountingPin, J4 Conn_01x26_MountingPin, J5 Conn_01x03, Q1 AO3400A, Q2 AO3400A, Q3 AO3400A, SW1 SW_Push, SW2 SW_Push, SW3 SKRTLAE010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

Commit message: gerbers
Parts:
- R42: value 10m -> WW25WR010FTL; footprint Resistor_SMD:R_0402_1005Metric -> linea:R2512; moved to B.Cu
- moved R42 8.74 mm to (81.4, 148.7)
Connections:
- R42 pad 1: +BATT -> Net-(U16-EN)
- R42 pad 2: Net-(U16-EN) -> +BATT
Routing:
- net +BATT: track 28.3 -> 41.5 mm, vias 1 -> 2
- net Net-(U16-EN): track 16.4 -> 18.5 mm
- net GND: vias 167 -> 169
