File: hardware/touchpad/touchpad.kicad_pcb (KiCad board)
At the start: 2 copper layers, 194.2 x 134.1 mm, 187 parts, among them J1 Conn_01x26_MountingPin, J10 Conn_02x03_Odd_Even, J100 Conn_02x03_Odd_Even, J101 Conn_02x03_Odd_Even, J102 Conn_02x03_Odd_Even, J103 Conn_02x03_Odd_Even, J104 Conn_02x03_Odd_Even, J105 Conn_02x03_Odd_Even, J106 Conn_02x03_Odd_Even, J107 Conn_02x03_Odd_Even, J108 Conn_02x03_Odd_Even, J109 Conn_02x03_Odd_Even, J11 Conn_02x03_Odd_Even, J110 Conn_02x03_Odd_Even, J111 Conn_02x03_Odd_Even, J112 Conn_02x03_Odd_Even, J113 Conn_02x03_Odd_Even, J114 Conn_02x03_Odd_Even, J115 Conn_02x03_Odd_Even, J116 Conn_02x03_Odd_Even, J117 Conn_02x03_Odd_Even, J118 Conn_02x03_Odd_Even, J119 Conn_02x03_Odd_Even, J12 Conn_02x03_Odd_Even, J120 Conn_02x03_Odd_Even, J121 Conn_02x03_Odd_Even, J122 Conn_02x03_Odd_Even, J123 Conn_02x03_Odd_Even, J124 Conn_02x03_Odd_Even, J125 Conn_02x03_Odd_Even, J126 Conn_02x03_Odd_Even, J127 Conn_02x03_Odd_Even, J128 Conn_02x03_Odd_Even, J129 Conn_02x03_Odd_Even, J13 Conn_02x03_Odd_Even, J130 Conn_02x03_Odd_Even, J131 Conn_02x03_Odd_Even, J132 Conn_02x03_Odd_Even, J133 Conn_02x03_Odd_Even, J134 Conn_02x03_Odd_Even, J135 Conn_02x03_Odd_Even, J136 Conn_02x03_Odd_Even, J137 Conn_02x03_Odd_Even, J138 Conn_02x03_Odd_Even, J139 Conn_02x03_Odd_Even, J14 Conn_02x03_Odd_Even, J140 Conn_02x03_Odd_Even, J141 Conn_02x03_Odd_Even, J142 Conn_02x03_Odd_Even, J143 Conn_02x03_Odd_Even, J144 Conn_02x03_Odd_Even, J145 Conn_02x03_Odd_Even, J146 Conn_02x03_Odd_Even, J147 Conn_02x03_Odd_Even, J148 Conn_02x03_Odd_Even, J149 Conn_02x03_Odd_Even, J15 Conn_02x03_Odd_Even, J150 Conn_02x03_Odd_Even, J151 Conn_02x03_Odd_Even, J152 Conn_02x03_Odd_Even, J153 Conn_02x03_Odd_Even, J154 Conn_02x03_Odd_Even, J155 Conn_02x03_Odd_Even, J156 Conn_02x03_Odd_Even, J157 Conn_02x03_Odd_Even, J158 Conn_02x03_Odd_Even, J159 Conn_02x03_Odd_Even, J16 Conn_02x03_Odd_Even, J160 Conn_02x03_Odd_Even, J161 Conn_02x03_Odd_Even, J162 Conn_02x03_Odd_Even, J163 Conn_02x03_Odd_Even, J164 Conn_02x03_Odd_Even, J165 Conn_02x03_Odd_Even, J166 Conn_02x03_Odd_Even, J167 Conn_02x03_Odd_Even, J168 Conn_02x03_Odd_Even, J169 Conn_02x03_Odd_Even, J17 Conn_02x03_Odd_Even, J170 Conn_02x03_Odd_Even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

Commit message: bunch o f stuff
Parts:
- moved J1 8.88 mm to (101.4, 15.9), turned to -90 degrees
- moved J2 4.50 mm to (60.0, 54.0), turned to 0 degrees
- moved J3 4.50 mm to (60.0, 85.3), turned to 0 degrees
Connections:
- J1 pad 1: /Y0 -> unconnected-(J1-Pin_1-Pad1)
- J1 pad 10: /Y7 -> /Y13
- J1 pad 11: /Y8 -> /Y12
- J1 pad 12: /Y9 -> /Y11
- J1 pad 13: GND -> /Y10
- J1 pad 14: /Y10 -> GND
- J1 pad 15: /Y11 -> /Y9
- J1 pad 16: /Y12 -> /Y8
- J1 pad 17: /Y13 -> /Y7
- J1 pad 18: GND -> /Y6
- J1 pad 19: /Y14 -> GND
- J1 pad 2: /Y1 -> unconnected-(J1-Pin_2-Pad2)
- J1 pad 20: /Y15 -> /Y5
- J1 pad 21: /Y16 -> /Y4
- J1 pad 22: /Y17 -> /Y3
- J1 pad 23: GND -> /Y2
- J1 pad 24: unconnected-(J1-Pin_24-Pad24) -> GND
- J1 pad 25: unconnected-(J1-Pin_25-Pad25) -> /Y1
- J1 pad 26: unconnected-(J1-Pin_26-Pad26) -> /Y0
- J1 pad 3: GND -> unconnected-(J1-Pin_3-Pad3)
- J1 pad 4: /Y2 -> GND
- J1 pad 5: /Y3 -> /Y17
- J1 pad 6: /Y4 -> /Y16
- J1 pad 7: /Y5 -> /Y15
- J1 pad 8: GND -> /Y14
- J1 pad 9: /Y6 -> GND
- J2 pad 1: /X0 -> unconnected-(J2-Pin_1-Pad1)
- J2 pad 10: /X7 -> /X13
- J2 pad 11: /X8 -> /X12
- J2 pad 12: /X9 -> /X11
- J2 pad 13: GND -> /X10
- J2 pad 14: /X10 -> GND
- J2 pad 15: /X11 -> /X9
- J2 pad 16: /X12 -> /X8
- J2 pad 17: /X13 -> /X7
- J2 pad 18: GND -> /X6
- J2 pad 19: /X14 -> GND
- J2 pad 2: /X1 -> /X19
- J2 pad 20: /X15 -> /X5
- J2 pad 21: /X16 -> /X4
- J2 pad 22: /X17 -> /X3
- J2 pad 23: GND -> /X2
- J2 pad 24: /X18 -> GND
- J2 pad 25: /X19 -> /X1
- J2 pad 26: unconnected-(J2-Pin_26-Pad26) -> /X0
- J2 pad 3: GND -> /X18
- J2 pad 4: /X2 -> GND
- J2 pad 5: /X3 -> /X17
- J2 pad 6: /X4 -> /X16
- J2 pad 7: /X5 -> /X15
- J2 pad 8: GND -> /X14
- J2 pad 9: /X6 -> GND
- J3 pad 1: /X20 -> unconnected-(J3-Pin_1-Pad1)
- J3 pad 10: /X27 -> unconnected-(J3-Pin_10-Pad10)
- J3 pad 13: GND -> unconnected-(J3-Pin_13-Pad13)
- J3 pad 14: unconnected-(J3-Pin_14-Pad14) -> GND
- J3 pad 17: unconnected-(J3-Pin_17-Pad17) -> /X27
- J3 pad 18: unconnected-(J3-Pin_18-Pad18) -> /X26
- J3 pad 19: unconnected-(J3-Pin_19-Pad19) -> GND
- J3 pad 2: /X21 -> unconnected-(J3-Pin_2-Pad2)
- J3 pad 20: unconnected-(J3-Pin_20-Pad20) -> /X25
- J3 pad 21: unconnected-(J3-Pin_21-Pad21) -> /X24
- J3 pad 22: unconnected-(J3-Pin_22-Pad22) -> /X23
- J3 pad 23: unconnected-(J3-Pin_23-Pad23) -> /X22
- J3 pad 24: unconnected-(J3-Pin_24-Pad24) -> GND
- J3 pad 25: unconnected-(J3-Pin_25-Pad25) -> /X21
- J3 pad 26: unconnected-(J3-Pin_26-Pad26) -> /X20
- J3 pad 3: GND -> unconnected-(J3-Pin_3-Pad3)
- J3 pad 4: /X22 -> unconnected-(J3-Pin_4-Pad4)
- J3 pad 5: /X23 -> unconnected-(J3-Pin_5-Pad5)
- J3 pad 6: /X24 -> unconnected-(J3-Pin_6-Pad6)
- J3 pad 7: /X25 -> unconnected-(J3-Pin_7-Pad7)
- J3 pad 8: GND -> unconnected-(J3-Pin_8-Pad8)
- J3 pad 9: /X26 -> unconnected-(J3-Pin_9-Pad9)
Routing:
- net GND: track 2517.6 -> 2526.9 mm
- net /Y5: track 198.2 -> 204.0 mm
- net /Y6: track 205.1 -> 211.0 mm
- net /Y7: track 211.8 -> 217.6 mm
- net /Y3: track 185.0 -> 190.7 mm
- net /Y4: track 191.7 -> 197.4 mm
- net /Y2: track 178.5 -> 184.2 mm
- net /Y0: track 164.8 -> 169.8 mm
- net /Y17: track 304.2 -> 299.2 mm
- net /Y1: track 171.6 -> 176.5 mm
- net /Y16: track 285.6 -> 280.9 mm
- net /Y11: track 240.3 -> 244.2 mm
- net /Y8: track 220.5 -> 224.4 mm
- net /Y10: track 233.8 -> 237.7 mm
- net /Y9: track 226.9 -> 230.8 mm
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Other:
- board size 194.2 x 134.1 mm -> 194.2 x 134.4 mm
